File: v1.0/schematics/eagle/vca/vca.sch (EAGLE design)
At the start: 20 parts, among them IC1 TL072P, J1 WAVE IN, J2 TRIGGER IN, J3 WAVE OUT, Q1 2N3417, Q2 2N3417, Q3 2N3417, Q4 2N3417, Q5 2N3906

Commit message: Updated VCA schem. Added VCF Diode Ladder
Parts:
- R2: value 330 -> 10K
- R5: value 330 -> 390
Changed lines of the file:
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@@
 <part name="J3" library="_common" deviceset="JACK-M" device="" value="WAVE OUT"/>
 <part name="R1" library="_common" deviceset="R" device="0309/10" value="10K"/>
-<part name="R2" library="_common" deviceset="R" device="0309/10" value="330"/>
+<part name="R2" library="_common" deviceset="R" device="0309/10" value="10K"/>
 <part name="R3" library="_common" deviceset="R" device="0309/10" value="2.2K"/>
 <part name="R4" library="_common" deviceset="R" device="0309/10" value="2.2K"/>
-<part name="R5" library="_common" deviceset="R" device="0309/10" value="330"/>
+<part name="R5" library="_common" deviceset="R" device="0309/10" value="390"/>
 <part name="R6" library="_common" deviceset="R" device="0309/10" value="10K"/>
 <part name="R7" library="_common" deviceset="R" device="0309/10" value="1K"/>
