File: v1.0/schematics/eagle/dlp.2-channel-mixer.v1.0.sch (EAGLE design)
At the start: 25 parts, among them IC1 TL082P, IC2 TL082P, J1 CH1-IN, J2 CH2-IN, J3 CH3-IN, J4 MIX-OUT, J5 CH3-OUT

Commit message: Created v2 of Midi2CV which serves MIDI channels 1 through 4 Updated out 2 name on mixer to indicate inverted out Regenerated vco pdf
Parts:
- J5: value CH3-OUT -> CH3-INV-OUT
Changed lines of the file:
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@@
 <?xml version="1.0" encoding="utf-8"?>
 <!DOCTYPE eagle SYSTEM "eagle.dtd">
-<eagle version="6.1">
+<eagle version="6.5.0">
 <drawing>
 <settings>
@@
 <setting verticaltext="up"/>
 </settings>
-<grid distance="0.1" unitdist="inch" unit="inch" style="lines" multiple="1" display="yes" altdistance="0.01" altunitdist="inch" altunit="inch"/>
+<grid distance="0.1" unitdist="inch" unit="inch" style="lines" multiple="1" display="no" altdistance="0.01" altunitdist="inch" altunit="inch"/>
 <layers>
 <layer number="1" name="Top" color="4" fill="1" visible="no" active="no"/>
@@
 <part name="J3" library="_common" deviceset="JACK-M" device="" value="CH3-IN"/>
 <part name="J4" library="_common" deviceset="JACK-M" device="" value="MIX-OUT"/>
-<part name="J5" library="_common" deviceset="JACK-M" device="" value="CH3-OUT"/>
+<part name="J5" library="_common" deviceset="JACK-M" device="" value="CH3-INV-OUT"/>
 <part name="C1" library="_common" deviceset="CE-US" device="E2-5" value="4.7μF"/>
 <part name="C2" library="_common" deviceset="CE-US" device="E2-5" value="4.7μF"/>
