File: v1.0/schematics/eagle/midi2cv/midi2cv.v2.sch (EAGLE design)
At the start: 28 parts, among them IC1 PIC18F2431DIP, IC2 TL084P, J1 CV MOD OUT, J2 CV VEL OUT, J3 CV PITCH OUT, J4 CV GATE OUT, Q1 20MHz

Commit message: Created v2 of Midi2CV which serves MIDI channels 1 through 4 Updated out 2 name on mixer to indicate inverted out Regenerated vco pdf
Parts:
- added C10, C11: 4.7uF, _common:CE-USE2-5
- added IC3: TL084P, _common:TL084P
- added IC4: TL082P, _common:TL082P
- added J10: GATE4 OUT, _common:JACK-M
- added J5: MOD2 OUT, _common:JACK-M
- added J6: VEL2 OUT, _common:JACK-M
- added J7: GATE1 OUT, _common:JACK-M
- added J8: GATE2 OUT, _common:JACK-M
- added J9: GATE3 OUT, _common:JACK-M
- added R10, R11, R12, R13, R8, R9: 390, _common:R0309/10
- added R14, R15, R16, R17, R18, R19, R20, R21, R22, R23: 1K, _common:R0309/10
- J1: value CV MOD OUT -> PITCH2 OUT
- J2: value CV VEL OUT -> MOD1 OUT
- J3: value CV PITCH OUT -> VEL1 OUT
- J4: value CV GATE OUT -> PITCH1 OUT
Connections:
- new net N$20: IC1.RB4/KBI0/PWM5, R8.1
- new net N$21: IC1.RB5/KBI1/PWM4/PGM, R9.1
- new net N$22: IC4A.-IN, IC4A.OUT, R15.1
- new net N$23: IC4B.-IN, IC4B.OUT, R16.1
- new net N$24: C11.+, IC4A.+IN, R9.2
- new net N$25: C10.+, IC4B.+IN, R8.2
- new net N$26: IC1.RA0/AN0, R10.2
- new net N$28: IC1.RA1/AN1, R11.2
- new net N$29: IC1.RA2/AN2/VREF-/CAP1/INDX, R12.2
- new net N$30: IC1.RA3/AN3/VREF+/CAP2/QEA, R13.2
- new net N$31: IC3D.-IN, IC3D.OUT, R23.2
- new net N$32: IC3D.+IN, R13.1
- new net N$33: IC3C.+IN, R12.1
- new net N$34: IC3A.+IN, R10.1
- new net N$35: IC3C.-IN, IC3C.OUT, R22.2
- new net N$36: IC3B.-IN, IC3B.OUT, R21.2
- new net N$37: IC3A.-IN, IC3A.OUT, R14.2
- new net N$38: J7.HOT, R14.1
- new net N$39: J8.HOT, R21.1
- new net N$40: J9.HOT, R22.1
- new net N$41: J10.HOT, R23.1
- new net N$42: J6.HOT, R15.2
- new net N$43: J5.HOT, R16.2
- new net N$44: J1.HOT, R17.2
- new net N$45: J2.HOT, R18.2
- new net N$46: J3.HOT, R19.2
- new net N$47: J4.HOT, R20.2
- new net N$5: IC3B.+IN, R11.1
- net +12V: now also IC3P.V+, IC4P.V+
- net -12V: now also IC3P.V-, IC4P.V-
- net 0V: now also C10.-, C11.-, J10.GND, J5.GND, J6.GND, J7.GND, J8.GND, J9.GND
- net N$16: now also IC1.RB3/PWM3; no longer IC1.RB4/KBI0/PWM5
- net N$17: now also IC1.RB2/PWM2; no longer IC1.RB3/PWM3
- net N$2: now also R17.1; no longer J1.HOT
- net N$3: now also R18.1; no longer J2.HOT
- net N$4: now also R19.1; no longer J3.HOT
- net N$7: now also R20.1; no longer J4.HOT
Other:
- note added: "MIDI to CV v2"
- note added: "Responsds to MIDI channels 1 through 4"
- note removed: "Built Feb 25, 2012"
- note removed: "MIDI to CV Converter"
- moved on the sheet: C2, C3, C4, C5, C6, C7, C8, C9, D2, IC2A, IC2B, IC2C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
