File: v1.0/schematics/eagle/bd/909.v1.sch (EAGLE design)
At the start: 80 parts, among them IC1 TL084P, IC2 TL082P, IC3 40106N, J1 OUT, J2 VELOCITY, J3 TRIGGER, Q1 2N3417, Q2 2N3906, Q3 2N3906, Q4 2N3417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

Commit message: Added schem for inital 909 kick module (omitted noise channel)
Parts:
- added C10: 0.33uF, _common:CC-US025-024X044
- added C9: 33nF, _common:CC-US025-024X044
- added D9: 1N4148, _common:1N4148
- added R43: 470K, _common:R0309/10
- C2: value 0.033uF -> 0.22uF
- C4: value 0.33uF (?) -> 0.033uF
- C5: value 0.33uF (?) -> 100pF
- C8: value 68nF -> 33nF
- R11: value 3.3K -> 2.2K
- R17: value 330K -> 270K
- R2: value 330K -> 320K
- R20: value 47K -> 2.2K
- R31: value 6.8K -> 5K
Connections:
- new net N$29: D9.A, J3.HOT
- net 0V: now also C10.1, R43.2
- net N$18: no longer R14.2
- net N$21: now also R43.1; no longer J3.HOT
- net N$22: now also R14.2
- net N$31: now also C9.2
- net N$33: now also C10.2
- net N$52: now also C9.1
Other:
- note added: "Currently omitted noise channel; may not include it for this version."
- note added: "Tailored for higher output, stable trigger, and sharper slope."
- note added: "which as based on the orignial TR-909 design."
- note added: "which was based on http://www.9090project.co.uk/"
- moved on the sheet: C6, C7, C8, D8, IC1D, IC3A, IC3B, J3, Q7, Q8, R13, R14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
