File: v2.0/schematics/eagle/vco/dlp.vco.dualosc.v1.1.main.sch (EAGLE design)
At the start: 44 parts, among them IC1 NTE912P, IC2 TL074P, IC3 TL074P, Q1 2N3417, Q2 2N3417, Q3 2N3906

Commit message: Added inital board for main schem (no real layout applied)
Parts:
- C1: value 0.01μF -> 0.01uF
- C5, C6: value 10μF -> 10uF
- JP2: value PANEL -> TO.PANEL; device pinhead:PINHD-2X10 -> pinhead:PINHD-1X10
Connections:
- net +12V: now also JP2.3; no longer JP2.5, JP2.6
- net -12V: no longer JP2.2
- net 0V: now also JP2.2; no longer JP2.3, JP2.4
- net N$EXP1: now also JP2.4; no longer JP2.7
- net N$OSC.OUT1: now also JP2.10; no longer JP2.19
- net N$PWM1: now also JP2.5; no longer JP2.9
- net N$SQ.LVL1A: now also JP2.8; no longer JP2.15
- net N$SQ.LVL1B: now also JP2.9; no longer JP2.17
- net N$SW.LVL1A: now also JP2.6; no longer JP2.11
- net N$SW.LVL1B: now also JP2.7; no longer JP2.13
Changed lines of the file:
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@@
 <part name="P+1" library="supply1" deviceset="+12V" device=""/>
 <part name="GND2" library="supply1" deviceset="0V" device=""/>
-<part name="C1" library="_common" deviceset="CC-US" device="025-024X044" value="0.01μF"/>
+<part name="C1" library="_common" deviceset="CC-US" device="025-024X044" value="0.01uF"/>
 <part name="IC1" library="_common" deviceset="NTE912" device="P"/>
 <part name="GND3" library="supply1" deviceset="0V" device=""/>
@@
 <part name="V/OCT1" library="rcl" deviceset="R-TRIMM" device="3296Y" value="100"/>
 <part name="HF-TRIM1" library="rcl" deviceset="R-TRIMM" device="3296Y" value="1M"/>
-<part name="C5" library="_common" deviceset="CE-US" device="E2-5" value="10μF"/>
-<part name="C6" library="_common" deviceset="CE-US" device="E2-5" value="10μF"/>
+<part name="C5" library="_common" deviceset="CE-US" device="E2-5" value="10uF"/>
+<part name="C6" library="_common" deviceset="CE-US" device="E2-5" value="10uF"/>
 <part name="R17" library="_common" deviceset="R" device="0309/10" value="22K"/>
 <part name="R18" library="_common" deviceset="R" device="0309/10" value="22K"/>
@@
 <part name="GND5" library="supply1" deviceset="0V" device=""/>
 <part name="GND9" library="supply1" deviceset="0V" device=""/>
-<part name="JP2" library="pinhead" deviceset="PINHD-2X10" device="" value="PANEL"/>
 <part name="GND14" library="supply1" deviceset="0V" device=""/>
-<part name="GND15" library="supply1" deviceset="0V" device=""/>
-<part name="P-9" library="supply1" deviceset="-12V" device=""/>
 <part name="P-10" library="supply1" deviceset="-12V" device=""/>
-<part name="P+10" library="supply1" deviceset="+12V" device=""/>
 <part name="P+11" library="supply1" deviceset="+12V" device=""/>
+<part name="JP2" library="pinhead" deviceset="PINHD-1X10" device="" value="TO.PANEL"/>
 </parts>
 <sheets>
@@
 headers.
 The next version will have a 2nd duplicated OSC.</text>
-<frame x1="-93.98" y1="-121.92" x2="215.9" y2="109.22" columns="8" rows="5" layer="91"/>
+<frame x1="-78.74" y1="-76.2" x2="210.82" y2="104.14" columns="8" rows="5" layer="91"/>
 </plain>
 <instances>
@@
 <instance part="GND5" gate="1" x="12.7" y="-58.42"/>
 <instance part="GND9" gate="1" x="48.26" y="-58.42"/>
-<instance part="JP2" gate="A" x="109.22" y="-43.18" rot="R180"/>
-<instance part="GND14" gate="1" x="124.46" y="-55.88"/>
-<instance part="GND15" gate="1" x="91.44" y="-55.88"/>
-<instance part="P-9" gate="1" x="96.52" y="-60.96"/>
-<instance part="P-10" gate="1" x="119.38" y="-60.96"/>
-<instance part="P+10" gate="1" x="86.36" y="-43.18" rot="MR0"/>
-<instance part="P+11" gate="1" x="137.16" y="-43.18" rot="MR0"/>
+<instance part="GND14" gate="1" x="88.9" y="-53.34"/>
+<instance part="P-10" gate="1" x="81.28" y="-58.42"/>
+<instance part="P+11" gate="1" x="96.52" y="-45.72" rot="MR0"/>
+<instance part="JP2" gate="A" x="68.58" y="-43.18" rot="R180"/>
 </instances>
 <busses>
@@
 </segment>
 <segment>
-<pinref part="JP2" gate="A" pin="4"/>
-<wire x1="104.14" y1="-50.8" x2="91.44" y2="-50.8" width="0.1524" layer="91"/>
-<pinref part="GND15" gate="1" pin="0V"/>
-<wire x1="91.44" y1="-50.8" x2="91.44" y2="-53.34" width="0.1524" layer="91"/>
-</segment>
-<segment>
-<pinref part="JP2" gate="A" pin="3"/>
-<wire x1="111.76" y1="-50.8" x2="124.46" y2="-50.8" width="0.1524" layer="91"/>
+<wire x1="71.12" y1="-50.8" x2="88.9" y2="-50.8" width="0.1524" layer="91"/>
 <pinref part="GND14" gate="1" pin="0V"/>
-<wire x1="124.46" y1="-50.8" x2="124.46" y2="-53.34" width="0.1524" layer="91"/>
+<pinref part="JP2" gate="A" pin="2"/>
 </segment>
 </net>
@@
 </segment>
 <segment>
-<pinref part="JP2" gate="A" pin="5"/>
-<wire x1="111.76" y1="-48.26" x2="137.16" y2="-48.26" width="0.1524" layer="91"/>
+<wire x1="71.12" y1="-48.26" x2="96.52" y2="-48.26" width="0.1524" layer="91"/>
 <pinref part="P+11" gate="1" pin="+12V"/>
-<wire x1="137.16" y1="-48.26" x2="137.16" y2="-45.72" width="0.1524" layer="91"/>
-</segment>
-<segment>
-<pinref part="JP2" gate="A" pin="6"/>
-<wire x1="104.14" y1="-48.26" x2="86.36" y2="-48.26" width="0.1524" layer="91"/>
-<pinref part="P+10" gate="1" pin="+12V"/>
-<wire x1="86.36" y1="-48.26" x2="86.36" y2="-45.72" width="0.1524" layer="91"/>
+<pinref part="JP2" gate="A" pin="3"/>
 </segment>
 </net>
@@
 </segment>
 <segment>
-<pinref part="JP2" gate="A" pin="2"/>
-<wire x1="104.14" y1="-53.34" x2="96.52" y2="-53.34" width="0.1524" layer="91"/>
-<pinref part="P-9" gate="1" pin="-12V"/>
-<wire x1="96.52" y1="-53.34" x2="96.52" y2="-58.42" width="0.1524" layer="91"/>
-</segment>
-<segment>
+<wire x1="71.12" y1="-53.34" x2="81.28" y2="-53.34" width="0.1524" layer="91"/>
+<pinref part="P-10" gate="1" pin="-12V"/>
+<wire x1="81.28" y1="-53.34" x2="81.28" y2="-55.88" width="0.1524" layer="91"/>
 <pinref part="JP2" gate="A" pin="1"/>
-<wire x1="111.76" y1="-53.34" x2="119.38" y2="-53.34" width="0.1524" layer="91"/>
-<pinref part="P-10" gate="1" pin="-12V"/>
-<wire x1="119.38" y1="-53.34" x2="119.38" y2="-58.42" width="0.1524" layer="91"/>
 </segment>
 </net>
@@
 <net name="N$EXP1" class="0">
 <segment>
-<wire x1="139.7" y1="-40.64" x2="132.08" y2="-40.64" width="0.1524" layer="91"/>
-<wire x1="132.08" y1="-40.64" x2="132.08" y2="-45.72" width="0.1524" layer="91"/>
-<wire x1="132.08" y1="-45.72" x2="111.76" y2="-45.72" width="0.1524" layer="91"/>
-<label x="139.7" y="-40.64" size="1.778" layer="95"/>
-<pinref part="JP2" gate="A" pin="7"/>
+<wire x1="78.74" y1="-45.72" x2="71.12" y2="-45.72" width="0.1524" layer="91"/>
+<label x="78.74" y="-45.72" size="1.778" layer="95"/>
+<pinref part="JP2" gate="A" pin="4"/>
 </segment>
 <segment>
@@
 <net name="N$PWM1" class="0">
 <segment>
-<pinref part="JP2" gate="A" pin="9"/>
-<wire x1="111.76" y1="-43.18" x2="129.54" y2="-43.18" width="0.1524" layer="91"/>
-<wire x1="129.54" y1="-43.18" x2="129.54" y2="-38.1" width="0.1524" layer="91"/>
-<wire x1="129.54" y1="-38.1" x2="139.7" y2="-38.1" width="0.1524" layer="91"/>
-<label x="139.7" y="-38.1" size="1.778" layer="95"/>
+<wire x1="71.12" y1="-43.18" x2="78.74" y2="-43.18" width="0.1524" layer="91"/>
+<label x="78.74" y="-43.18" size="1.778" layer="95"/>
+<pinref part="JP2" gate="A" pin="5"/>
 </segment>
 <segment>
@@
 <net name="N$SW.LVL1A" class="0">
 <segment>
-<pinref part="JP2" gate="A" pin="11"/>
-<wire x1="111.76" y1="-40.64" x2="127" y2="-40.64" width="0.1524" layer="91"/>
-<wire x1="127" y1="-40.64" x2="127" y2="-35.56" width="0.1524" layer="91"/>
-<wire x1="127" y1="-35.56" x2="139.7" y2="-35.56" width="0.1524" layer="91"/>
-<label x="139.7" y="-35.56" size="1.778" layer="95"/>
+<wire x1="71.12" y1="-40.64" x2="78.74" y2="-40.64" width="0.1524" layer="91"/>
+<label x="78.74" y="-40.64" size="1.778" layer="95"/>
+<pinref part="JP2" gate="A" pin="6"/>
 </segment>
 <segment>
@@
 <net name="N$SW.LVL1B" class="0">
 <segment>
-<pinref part="JP2" gate="A" pin="13"/>
-<wire x1="111.76" y1="-38.1" x2="124.46" y2="-38.1" width="0.1524" layer="91"/>
-<wire x1="124.46" y1="-38.1" x2="124.46" y2="-33.02" width="0.1524" layer="91"/>
-<wire x1="124.46" y1="-33.02" x2="139.7" y2="-33.02" width="0.1524" layer="91"/>
-<label x="139.7" y="-33.02" size="1.778" layer="95"/>
+<wire x1="71.12" y1="-38.1" x2="78.74" y2="-38.1" width="0.1524" layer="91"/>
+<label x="78.74" y="-38.1" size="1.778" layer="95"/>
+<pinref part="JP2" gate="A" pin="7"/>
 </segment>
 <segment>
@@
 <net name="N$SQ.LVL1A" class="0">
 <segment>
-<pinref part="JP2" gate="A" pin="15"/>
-<wire x1="111.76" y1="-35.56" x2="121.92" y2="-35.56" width="0.1524" layer="91"/>
-<wire x1="121.92" y1="-35.56" x2="121.92" y2="-30.48" width="0.1524" layer="91"/>
-<wire x1="121.92" y1="-30.48" x2="139.7" y2="-30.48" width="0.1524" layer="91"/>
-<label x="139.7" y="-30.48" size="1.778" layer="95"/>
+<wire x1="71.12" y1="-35.56" x2="78.74" y2="-35.56" width="0.1524" layer="91"/>
+<label x="78.74" y="-35.56" size="1.778" layer="95"/>
+<pinref part="JP2" gate="A" pin="8"/>
 </segment>
 <segment>
@@
 <net name="N$SQ.LVL1B" class="0">
 <segment>
-<pinref part="JP2" gate="A" pin="17"/>
-<wire x1="111.76" y1="-33.02" x2="119.38" y2="-33.02" width="0.1524" layer="91"/>
-<wire x1="119.38" y1="-33.02" x2="119.38" y2="-27.94" width="0.1524" layer="91"/>
-<wire x1="119.38" y1="-27.94" x2="139.7" y2="-27.94" width="0.1524" layer="91"/>
-<label x="139.7" y="-27.94" size="1.778" layer="95"/>
+<wire x1="71.12" y1="-33.02" x2="78.74" y2="-33.02" width="0.1524" layer="91"/>
+<label x="78.74" y="-33.02" size="1.778" layer="95"/>
+<pinref part="JP2" gate="A" pin="9"/>
 </segment>
 <segment>
@@
 <net name="N$OSC.OUT1" class="0">
 <segment>
-<pinref part="JP2" gate="A" pin="19"/>
-<wire x1="111.76" y1="-30.48" x2="116.84" y2="-30.48" width="0.1524" layer="91"/>
-<wire x1="116.84" y1="-30.48" x2="116.84" y2="-25.4" width="0.1524" layer="91"/>
-<wire x1="116.84" y1="-25.4" x2="139.7" y2="-25.4" width="0.1524" layer="91"/>
-<label x="139.7" y="-25.4" size="1.778" layer="95"/>
-</segment>
-<segment>
+<wire x1="71.12" y1="-30.48" x2="78.74" y2="-30.48" width="0.1524" layer="91"/>
+<label x="78.74" y="-30.48" size="1.778" layer="95"/>
+<pinref part="JP2" gate="A" pin="10"/>
+</segment>
+<segment>
