File: v1.0/schematics/eagle/psu/psu-12v.sch (EAGLE design)
At the start: 16 parts, among them IC1 7812T, IC2 7912T, IC3 7805T

Commit message: Update component names on board layout Reverse cap polarity on v1.0 psu schem
Connections:
- removed net N$4: C2.+, D2.A, IC2.VI
- new net N$5: C2.-, D2.A, IC2.VI
- net +12V: now also C3.+; no longer C3.-
- net +5V: now also C4.+; no longer C4.-
- net -12V: now also C5.-; no longer C5.+
- net 0V: now also C1.-, C2.+, C3.-, C4.-, C5.+; no longer C1.+, C2.-, C3.+, C4.+, C5.-
- net N$3: now also C1.+; no longer C1.-
Other:
- moved on the sheet: C1, C2, C3, C4, C5
