File: v2.0/schematics/eagle/midi2cv.rev2/midi2cv.2.2.main.sch (EAGLE design)
At the start: 36 parts, among them IC1 PIC18F2431DIP, Q1 20MHz, X1 MAB5SH

Commit message: Updated version on schem and board to 2.2 Revised labels for GATE1..5 to match board layout and firmare
Connections:
- net GATE1: now also JP2.9, R5.2; no longer JP2.2, R1.1
- net GATE2: now also JP2.8, R4.1; no longer JP2.4, R2.1
- net GATE4: now also JP2.4, R2.1; no longer JP2.8, R4.1
- net GATE5: now also JP2.2, R1.1; no longer JP2.9, R5.2
Other:
- note added: "MIDI to CV v2.2 (Multi Mode) Either mode responds to all MIDI channels MODE0: Synth mode (switch closed) - CV1: PITCH - CV2: VEL - CV3: MOD (CC1) - GATE1: GATE - GATE2-5: CC2-5 > 63 MODE1: Drum mode (switch open) - Responds to C1, C#1, D1, D#1, E1 - CV1: VEL (C1) - CV2: VEL (C#1) - CV3: VEL (D1) - GATE1-5: GATE (C1 to E1)"
- note removed: "MIDI to CV v2.0 (Multi Mode) Either mode responds to all MIDI channels MODE0: Synth mode - CV1: PITCH - CV2: VEL - CV3: MOD (CC1) - GATE1: GATE - GATE2-5: CC2-5 > 63 MODE1: Drum mode - Responds to C1, C#1, D1, D#1, E1 - CV1: VEL (C1) - CV2: VEL (C#1) - CV3: VEL (D1) - GATE1-5: GATE (C1 to E1)"
Changed lines of the file:
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@@
 <?xml version="1.0" encoding="utf-8"?>
 <!DOCTYPE eagle SYSTEM "eagle.dtd">
-<eagle version="7.5.0">
+<eagle version="7.2.0">
 <drawing>
 <settings>
@@
 <sheet>
 <plain>
-<text x="137.16" y="93.98" size="1.778" layer="97">MIDI to CV v2.0 (Multi Mode)
+<text x="137.16" y="93.98" size="1.778" layer="97">MIDI to CV v2.2 (Multi Mode)
 Either mode responds to all MIDI channels
-MODE0: Synth mode
+MODE0: Synth mode (switch closed)
 - CV1: PITCH
 - CV2: VEL
@@
 - GATE1: GATE
 - GATE2-5: CC2-5 &gt; 63
-MODE1: Drum mode
+MODE1: Drum mode (switch open)
 - Responds to C1, C#1, D1, D#1, E1
 - CV1: VEL (C1)
@@
 </segment>
 </net>
-<net name="GATE1" class="0">
+<net name="GATE3" class="0">
+<segment>
+<pinref part="JP2" gate="A" pin="6"/>
+<wire x1="-10.16" y1="114.3" x2="-17.78" y2="114.3" width="0.1524" layer="91"/>
+<label x="-22.86" y="114.3" size="1.778" layer="95"/>
+</segment>
+<segment>
+<pinref part="R3" gate="G$1" pin="1"/>
+<wire x1="-17.78" y1="73.66" x2="-20.32" y2="73.66" width="0.1524" layer="91"/>
+<label x="-25.4" y="73.66" size="1.778" layer="95"/>
+</segment>
+</net>
+<net name="CV2" class="0">
+<segment>
+<pinref part="JP2" gate="A" pin="13"/>
+<wire x1="-2.54" y1="124.46" x2="5.08" y2="124.46" width="0.1524" layer="91"/>
+<label x="5.08" y="124.46" size="1.778" layer="95"/>
+</segment>
+<segment>
+<pinref part="R11" gate="G$1" pin="2"/>
+<wire x1="147.32" y1="71.12" x2="149.86" y2="71.12" width="0.1524" layer="91"/>
+<label x="149.86" y="71.12" size="1.778" layer="95"/>
+</segment>
+</net>
+<net name="CV3" class="0">
+<segment>
+<pinref part="JP2" gate="A" pin="15"/>
+<wire x1="-2.54" y1="127" x2="5.08" y2="127" width="0.1524" layer="91"/>
+<label x="5.08" y="127" size="1.778" layer="95"/>
+</segment>
+<segment>
+<pinref part="R10" gate="G$1" pin="2"/>
+<wire x1="147.32" y1="78.74" x2="149.86" y2="78.74" width="0.1524" layer="91"/>
+<label x="149.86" y="78.74" size="1.778" layer="95"/>
+</segment>
+</net>
+<net name="CV1" class="0">
+<segment>
+<pinref part="JP2" gate="A" pin="11"/>
+<wire x1="5.08" y1="121.92" x2="-2.54" y2="121.92" width="0.1524" layer="91"/>
+<label x="5.08" y="121.92" size="1.778" layer="95"/>
+</segment>
+<segment>
+<pinref part="R12" gate="G$1" pin="2"/>
+<wire x1="147.32" y1="63.5" x2="149.86" y2="63.5" width="0.1524" layer="91"/>
+<label x="149.86" y="63.5" size="1.778" layer="95"/>
+</segment>
+</net>
+<net name="GATE5" class="0">
+<segment>
+<pinref part="R1" gate="G$1" pin="1"/>
+<wire x1="-17.78" y1="88.9" x2="-20.32" y2="88.9" width="0.1524" layer="91"/>
+<label x="-25.4" y="88.9" size="1.778" layer="95"/>
+</segment>
 <segment>
 <pinref part="JP2" gate="A" pin="2"/>
@@
 <label x="-22.86" y="109.22" size="1.778" layer="95"/>
 </segment>
-<segment>
-<pinref part="R1" gate="G$1" pin="1"/>
-<wire x1="-17.78" y1="88.9" x2="-20.32" y2="88.9" width="0.1524" layer="91"/>
-<label x="-25.4" y="88.9" size="1.778" layer="95"/>
-</segment>
-</net>
-<net name="GATE2" class="0">
+</net>
+<net name="GATE4" class="0">
+<segment>
+<pinref part="R2" gate="G$1" pin="1"/>
+<wire x1="-17.78" y1="81.28" x2="-20.32" y2="81.28" width="0.1524" layer="91"/>
+<label x="-25.4" y="81.28" size="1.778" layer="95"/>
+</segment>
 <segment>
 <pinref part="JP2" gate="A" pin="4"/>
@@
 <label x="-22.86" y="111.76" size="1.778" layer="95"/>
 </segment>
-<segment>
-<pinref part="R2" gate="G$1" pin="1"/>
-<wire x1="-17.78" y1="81.28" x2="-20.32" y2="81.28" width="0.1524" layer="91"/>
-<label x="-25.4" y="81.28" size="1.778" layer="95"/>
-</segment>
-</net>
-<net name="GATE3" class="0">
-<segment>
-<pinref part="JP2" gate="A" pin="6"/>
-<wire x1="-10.16" y1="114.3" x2="-17.78" y2="114.3" width="0.1524" layer="91"/>
-<label x="-22.86" y="114.3" size="1.778" layer="95"/>
-</segment>
-<segment>
-<pinref part="R3" gate="G$1" pin="1"/>
-<wire x1="-17.78" y1="73.66" x2="-20.32" y2="73.66" width="0.1524" layer="91"/>
-<label x="-25.4" y="73.66" size="1.778" layer="95"/>
-</segment>
-</net>
-<net name="GATE4" class="0">
+</net>
+<net name="GATE2" class="0">
+<segment>
+<pinref part="R4" gate="G$1" pin="1"/>
+<wire x1="-17.78" y1="66.04" x2="-20.32" y2="66.04" width="0.1524" layer="91"/>
+<label x="-25.4" y="66.04" size="1.778" layer="95"/>
+</segment>
 <segment>
 <pinref part="JP2" gate="A" pin="8"/>
@@
 <label x="-22.86" y="116.84" size="1.778" layer="95"/>
 </segment>
-<segment>
-<pinref part="R4" gate="G$1" pin="1"/>
-<wire x1="-17.78" y1="66.04" x2="-20.32" y2="66.04" width="0.1524" layer="91"/>
-<label x="-25.4" y="66.04" size="1.778" layer="95"/>
-</segment>
-</net>
-<net name="GATE5" class="0">
+</net>
+<net name="GATE1" class="0">
+<segment>
+<pinref part="R5" gate="G$1" pin="2"/>
+<wire x1="-17.78" y1="58.42" x2="-20.32" y2="58.42" width="0.1524" layer="91"/>
+<label x="-25.4" y="58.42" size="1.778" layer="95"/>
+</segment>
 <segment>
 <pinref part="JP2" gate="A" pin="9"/>
@@
 <label x="5.08" y="119.38" size="1.778" layer="95"/>
 </segment>
-<segment>
-<pinref part="R5" gate="G$1" pin="2"/>
-<wire x1="-17.78" y1="58.42" x2="-20.32" y2="58.42" width="0.1524" layer="91"/>
-<label x="-25.4" y="58.42" size="1.778" layer="95"/>
-</segment>
-</net>
-<net name="CV2" class="0">
-<segment>
-<pinref part="JP2" gate="A" pin="13"/>
-<wire x1="-2.54" y1="124.46" x2="5.08" y2="124.46" width="0.1524" layer="91"/>
-<label x="5.08" y="124.46" size="1.778" layer="95"/>
-</segment>
-<segment>
-<pinref part="R11" gate="G$1" pin="2"/>
-<wire x1="147.32" y1="71.12" x2="149.86" y2="71.12" width="0.1524" layer="91"/>
-<label x="149.86" y="71.12" size="1.778" layer="95"/>
-</segment>
-</net>
-<net name="CV3" class="0">
-<segment>
-<pinref part="JP2" gate="A" pin="15"/>
-<wire x1="-2.54" y1="127" x2="5.08" y2="127" width="0.1524" layer="91"/>
-<label x="5.08" y="127" size="1.778" layer="95"/>
-</segment>
-<segment>
-<pinref part="R10" gate="G$1" pin="2"/>
-<wire x1="147.32" y1="78.74" x2="149.86" y2="78.74" width="0.1524" layer="91"/>
-<label x="149.86" y="78.74" size="1.778" layer="95"/>
-</segment>
-</net>
-<net name="CV1" class="0">
-<segment>
-<pinref part="JP2" gate="A" pin="11"/>
-<wire x1="5.08" y1="121.92" x2="-2.54" y2="121.92" width="0.1524" layer="91"/>
-<label x="5.08" y="121.92" size="1.778" layer="95"/>
-</segment>
-<segment>
-<pinref part="R12" gate="G$1" pin="2"/>
-<wire x1="147.32" y1="63.5" x2="149.86" y2="63.5" width="0.1524" layer="91"/>
-<label x="149.86" y="63.5" size="1.778" layer="95"/>
-</segment>
-</net>
+</net>
