File: v2.0/schematics/eagle/dcy.vca/dcy.vca.v1.0.0.sch (EAGLE design)
At the start: 77 parts, among them IC1 TL072P, IC2 4001N, IC3 LM324N, IC4 TL074P, IC5 4001N, IC7 TL074P, Q1 2N3704, Q2 2N3704, Q3 2N3704, Q4 2N3704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

Commit message: Changed 10K to 390 on vca schem
Parts:
- R2: value 10K -> 390
Changed lines of the file:
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@@
 <parts>
 <part name="R1" library="_common" deviceset="R" device="0309/10" value="10K"/>
-<part name="R2" library="_common" deviceset="R" device="0309/10" value="10K"/>
+<part name="R2" library="_common" deviceset="R" device="0309/10" value="390"/>
 <part name="R3" library="_common" deviceset="R" device="0309/10" value="2.2K"/>
 <part name="R4" library="_common" deviceset="R" device="0309/10" value="2.2K"/>

Commit message: Added inital schem and board for quad.vca module. Added ota library for LM137000 Modified symbol for switched mono jacks Added 2N3904 and 7.5mm resistor to common.lbr
Parts:
- added D5: 1N4148, _common:1N4148
Connections:
- new net N$63: C3.+, D5.C, IC4B.+IN, RV1.2
- net N$17: now also D5.A; no longer C3.+, IC4B.+IN, RV1.2
Other:
- note added: "Need to test this, but i think all the dcy's need a diode here to prevent the cap drain through the op amp"
Changed lines of the file:
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@@
 <part name="GND46" library="supply1" deviceset="0V" device=""/>
 <part name="GND47" library="supply1" deviceset="0V" device=""/>
+<part name="D5" library="_common" deviceset="1N4148" device=""/>
 </parts>
 <sheets>
@@
 - Single VCA</text>
 <frame x1="-281.94" y1="-71.12" x2="93.98" y2="152.4" columns="8" rows="5" layer="91"/>
+<text x="-144.78" y="134.62" size="1.778" layer="91">Need to test this, but i think all the dcy's need a diode here to prevent the cap drain through the op amp</text>
 </plain>
 <instances>
@@
 <instance part="GND46" gate="1" x="76.2" y="-38.1"/>
 <instance part="GND47" gate="1" x="33.02" y="-40.64"/>
+<instance part="D5" gate="G$1" x="-152.4" y="119.38"/>
 </instances>
 <busses>
@@
 <wire x1="-172.72" y1="111.76" x2="-157.48" y2="111.76" width="0.1524" layer="91"/>
 <wire x1="-157.48" y1="111.76" x2="-157.48" y2="119.38" width="0.1524" layer="91"/>
-<pinref part="IC4" gate="B" pin="+IN"/>
-<wire x1="-157.48" y1="119.38" x2="-149.86" y2="119.38" width="0.1524" layer="91"/>
-<pinref part="C3" gate="G$1" pin="+"/>
-<wire x1="-149.86" y1="119.38" x2="-139.7" y2="119.38" width="0.1524" layer="91"/>
-<wire x1="-139.7" y1="119.38" x2="-134.62" y2="119.38" width="0.1524" layer="91"/>
-<wire x1="-149.86" y1="119.38" x2="-149.86" y2="116.84" width="0.1524" layer="91"/>
-<pinref part="RV1" gate="G$1" pin="2"/>
-<wire x1="-139.7" y1="119.38" x2="-139.7" y2="109.22" width="0.1524" layer="91"/>
+<pinref part="D5" gate="G$1" pin="A"/>
+<wire x1="-157.48" y1="119.38" x2="-154.94" y2="119.38" width="0.1524" layer="91"/>
 <junction x="-157.48" y="119.38"/>
-<junction x="-139.7" y="119.38"/>
-<junction x="-149.86" y="119.38"/>
 </segment>
 </net>
@@
 </segment>
 </net>
+<net name="N$63" class="0">
+<segment>
+<pinref part="IC4" gate="B" pin="+IN"/>
+<pinref part="RV1" gate="G$1" pin="2"/>
+<pinref part="C3" gate="G$1" pin="+"/>
+<wire x1="-149.86" y1="119.38" x2="-149.86" y2="116.84" width="0.1524" layer="91"/>
+<wire x1="-149.86" y1="119.38" x2="-139.7" y2="119.38" width="0.1524" layer="91"/>
+<wire x1="-139.7" y1="119.38" x2="-139.7" y2="109.22" width="0.1524" layer="91"/>
+<junction x="-139.7" y="119.38"/>
+<wire x1="-139.7" y1="119.38" x2="-134.62" y2="119.38" width="0.1524" layer="91"/>
+<pinref part="D5" gate="G$1" pin="C"/>
+<junction x="-149.86" y="119.38"/>
+</segment>
+</net>
+<net name="N$64" class="0">
+<segment>
+<wire x1="-152.4" y1="124.46" x2="-144.78" y2="132.08" width="0.1524" layer="91"/>
+</segment>
+</net>
