File: v2.0/schematics/eagle/quad.vca/dual.vca.pnl.brd (EAGLE design)
At the start: 100 x 80 mm, 66 parts, among them IC1 TL084P, IC2 LM13700N, J1 CV2-A, J2 CV1-A, J3 IN-A, J4 OUT-A, J5 CV2-B, J6 CV1-B, J7 IN-B, J8 OUT-B, Q1 2N3904, Q2 2N3906, Q3 2N3904, Q4 2N3906

Commit message: Completed VCA main and panel schems (quad vca is now dual) Updated exclusion zones on mono jack
Parts:
- removed BIAS-A, BIAS-B: 100K, pot:PT-10S
- removed CV2ATT-A, CV2ATT-B, CVOFFS-A, CVOFFS-B: 100K, _common:R-VAR
- removed FEED-A, FEED-B: 2K, pot:PT-10S
- removed IC1: TL084P, linear:DIL14
- removed IC2: LM13700N, ota:DIL16
- removed JP2: LOG/LIN, pinhead:1X03
- removed Q1, Q3: 2N3904, _common:TO92
- removed Q2, Q4: 2N3906, _common:TO92
- removed R1, R17, R21, R24, R26, R3, R31, R40, R44, R8: 100K, resistor:0207/7
- removed R11, R34: 120K, resistor:0207/7
- removed R12, R35: 2.2M, resistor:0207/7
- removed R13, R23, R36, R46: 20K, resistor:0207/7
- removed R14, R37: 470K, resistor:0207/7
- removed R15, R38: 47K, resistor:0207/7
- removed R16, R27, R32, R39, R4, R9: 2K, resistor:0207/7
- removed R18, R41: 470, resistor:0207/7
- removed R19, R42: 4.7K, resistor:0207/7
- removed R22, R45: 30K, resistor:0207/7
- removed R30, R7: 150, resistor:0207/7
- added JP3: IO-B, pinhead:1X05
- JP1: value LOG/LIN -> IO-A; device pinhead:1X03 -> pinhead:1X05
- moved R43 309.3 mm to (60.3, 37.5), turned to 180 degrees
- moved R28 273.5 mm to (67.9, 1.91)
- moved J5 256.3 mm to (51.4, 23.5)
- moved R25 249.4 mm to (57.8, 1.91)
- moved J8 235.4 mm to (67.9, 23.5)
- moved J6 225.3 mm to (51.4, 6.99)
- moved J7 225.3 mm to (67.9, 6.99)
- moved JP1 209.7 mm to (1.91, 19.7), turned to 90 degrees
- moved J1 172.8 mm to (15.9, 23.5)
- moved R20 167.9 mm to (14.6, 37.5)
- moved R5 113.7 mm to (17.1, 1.91), turned to 180 degrees
- moved R2 52.9 mm to (6.99, 1.91), turned to 180 degrees
- moved J3 50.7 mm to (32.4, 6.99)
- moved J4 50.7 mm to (32.4, 23.5)
- moved J2 32.5 mm to (15.9, 6.99)
Connections:
- removed net +12V: BIAS-A.E, BIAS-B.E, CVOFFS-A.R2, CVOFFS-B.R2, IC1.4, IC2.11, Q1.3, Q3.3, R14.2, R17.2, R26.2, R3.2, R37.2, R40.2
- removed net -12V: BIAS-A.A, BIAS-B.A, CVOFFS-A.R1, CVOFFS-B.R1, IC1.11, IC2.6, R11.1, R19.1, R23.1, R34.1, R42.1, R46.1
- removed net N$10: JP1.1, R13.1
- removed net N$12: FEED-A.E, FEED-A.S, IC2.3, R5.2
- removed net N$13: IC2.8, R19.2, R20.1
- removed net N$14: BIAS-A.S, R12.1
- removed net N$15: IC2.5, IC2.7, R12.2, R14.1, R15.2
- removed net N$17: CV2ATT-A.VAR, R1.2
- removed net N$18: JP1.3, R22.1, R23.2
- removed net N$19: IC1.5, R17.1, R18.2
- removed net N$20: IC1.6, R16.2, R21.1
- removed net N$21: IC2.1, JP1.2
- removed net N$22: IC1.7, R21.2, R22.2
- removed net N$25: IC1.10, R26.1, R27.2
- removed net N$26: IC1.9, R24.1, R25.2, R31.2, R32.1
- removed net N$27: CVOFFS-B.VAR, R31.1
- removed net N$28: IC1.8, Q3.2, R32.2, R39.1
- removed net N$29: Q3.1, Q4.2, R34.2
- removed net N$30: Q4.1, R36.2
- removed net N$31: FEED-B.A, R30.2
- removed net N$33: FEED-B.E, FEED-B.S, IC2.14, R28.2
- removed net N$34: BIAS-B.S, R35.1
- removed net N$35: IC2.10, IC2.12, R35.2, R37.1, R38.2
- removed net N$36: IC2.9, R42.2, R43.1
- removed net N$38: CV2ATT-B.VAR, R24.2
- removed net N$39: IC1.12, R40.1, R41.2
- removed net N$40: IC1.13, R39.2, R44.1
- removed net N$41: IC1.14, R44.2, R45.2
- removed net N$42: JP2.1, R36.1
- removed net N$43: JP2.3, R45.1, R46.2
- removed net N$44: IC2.16, JP2.2
- removed net N$6: IC1.1, Q1.2, R16.1, R9.2
- net 0V: now also JP1.5, JP3.5; no longer CV2ATT-A.R1, CV2ATT-B.R1, IC2.13, IC2.4, Q2.3, Q4.3, R15.1, R18.1, R27.1, R30.1, R38.1, R4.1, R41.1, R7.1
- net N$16: now also JP1.1; no longer CV2ATT-A.R2
- net N$3: now also JP1.2, R2.2; no longer IC1.3, R3.1, R4.2
- net N$37: now also JP3.1; no longer CV2ATT-B.R2
- net N$4: now also JP1.3, R5.2; no longer IC1.2, R1.1, R2.2, R8.2, R9.1
- net N$5: now also JP1.4, R20.1; no longer CVOFFS-A.VAR, R8.1
- net N$7: now also JP3.2, R25.2; no longer Q1.1, Q2.2, R11.2
- net N$8: now also JP3.3, R28.2; no longer FEED-A.A, R7.2
- net N$9: now also JP3.4, R43.1; no longer Q2.1, R13.2
Routing:
- net 0V: track 0.00 -> 161.0 mm
- net N$37: track 0.00 -> 39.1 mm
- net N$4: track 0.00 -> 22.6 mm
- net N$7: track 0.00 -> 21.2 mm
- net N$5: track 0.00 -> 19.7 mm
- net N$8: track 0.00 -> 18.9 mm, vias 0 -> 1
- net N$9: track 0.00 -> 18.9 mm
- net N$2: track 0.00 -> 18.5 mm
- net N$23: track 0.00 -> 18.5 mm
- net N$16: track 0.00 -> 17.6 mm
- net N$24: track 0.00 -> 17.5 mm
- net N$3: track 0.00 -> 16.4 mm
- net N$32: track 0.00 -> 12.4 mm
- net N$1: track 0.00 -> 11.7 mm
- net N$11: track 0.00 -> 9.32 mm
Other:
- board size 100 x 80 mm -> 75.2 x 39.4 mm
