File: v2.0/schematics/eagle/quad.vca/dual.vca.main.sch (EAGLE design)
At the start: 66 parts, among them IC1 TL084P, IC2 LM13700N, J1 CV2-A, J2 CV1-A, J3 IN-A, J4 OUT-A, J5 CV2-B, J6 CV1-B, J7 IN-B, J8 OUT-B, Q1 2N3904, Q2 2N3906, Q3 2N3904, Q4 2N3906

Commit message: Completed VCA main and panel schems (quad vca is now dual) Updated exclusion zones on mono jack
Parts:
- removed J1: CV2-A, jacks:ACJM-MV35-2S
- removed J2: CV1-A, jacks:ACJM-MV35-2S
- removed J3: IN-A, jacks:ACJM-MV35-2S
- removed J4: OUT-A, jacks:ACJM-MV35-2S
- removed J5: CV2-B, jacks:ACJM-MV35-2S
- removed J6: CV1-B, jacks:ACJM-MV35-2S
- removed J7: IN-B, jacks:ACJM-MV35-2S
- removed J8: OUT-B, jacks:ACJM-MV35-2S
- removed R2, R25, R28, R5: 100K, resistor:R-US_0207/7
- removed R20, R43: 1K, resistor:R-US_0207/7
- added C1, C2, C3, C4: 0.1uF, _common:CC-US025-024X044
- added C5, C6: 10uF, _common:CE-USE2-5
- added JP3: IO-A, pinhead:PINHD-1X5
- added JP4: IO-B, pinhead:PINHD-1X5
- added JP5: PWR, pinhead:PINHD-2X8
Connections:
- removed net N$1: J2.P$2, J2.P$3, R2.1
- removed net N$11: J3.P$2, R5.1
- removed net N$12: FEED-A.E, FEED-A.S, IC2OTA1.IN_P, R5.2
- removed net N$13: IC2BUF1.E, R19.2, R20.1
- removed net N$16: CV2ATT-A.2, J1.P$2, J1.P$3
- removed net N$2: J4.P$2, J4.P$3, R20.2
- removed net N$23: J6.P$2, J6.P$3, R25.1
- removed net N$24: J8.P$2, J8.P$3, R43.2
- removed net N$26: IC1C.-IN, R24.1, R25.2, R31.2, R32.1
- removed net N$32: J7.P$2, R28.1
- removed net N$33: FEED-B.E, FEED-B.S, IC2OTA2.IN_P, R28.2
- removed net N$36: IC2BUF2.E, R42.2, R43.1
- removed net N$37: CV2ATT-B.2, J5.P$2, J5.P$3
- removed net N$4: IC1A.-IN, R1.1, R2.2, R8.2, R9.1
- new net CV1-A: IC1A.-IN, JP3.2, R1.1, R8.2, R9.1
- new net CV1-B: IC1C.-IN, JP4.2, R24.1, R31.2, R32.1
- new net CV2-A: CV2ATT-A.2, JP3.1
- new net CV2-B: CV2ATT-B.2, JP4.1
- new net IN-A: FEED-A.E, FEED-A.S, IC2OTA1.IN_P, JP3.3
- new net IN-B: FEED-B.E, FEED-B.S, IC2OTA2.IN_P, JP4.3
- new net OUT-A: IC2BUF1.E, JP3.4, R19.2
- new net OUT-B: IC2BUF2.E, JP4.4, R42.2
- net +12V: now also C1.1, C2.1, C5.+, JP5.10, JP5.9
- net -12V: now also C3.2, C4.2, C6.-, JP5.1, JP5.2
- net 0V: now also C1.2, C2.2, C3.1, C4.1, C5.-, C6.+, JP3.5, JP4.5, JP5.3, JP5.4, JP5.5, JP5.6, JP5.7, JP5.8; no longer J1.P$1, J2.P$1, J3.P$1, J3.P$3, J4.P$1, J5.P$1, J6.P$1, J7.P$1, J7.P$3, J8.P$1
Other:
- note added: "dual.vca.main.v2.0 Adapted from Ray Wilson's RJWSoft Dual Log/Linear VCA: http://www.musicfromouterspace.com/analogsynth_new/DUALVCA/DLLVCA001.html"
- note removed: "Adapted from Ray Wilson's RJWSoft Dual Log/Linear VCA: http://www.musicfromouterspace.com/analogsynth_new/DUALVCA/DLLVCA001.html"
- moved on the sheet: BIAS-A, BIAS-B, CV2ATT-A, CV2ATT-B, CVOFFS-A, CVOFFS-B, FEED-A, FEED-B, IC1A, IC1B, IC1C, IC1D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

Commit message: Replaced trim pots with tested fixed values. Corrected error in PNP transisitor connection
Connections:
- removed net N$30: Q4.E, R36.2
- removed net N$9: Q2.E, R13.2
- new net N$1: Q2.C, R13.2
- new net N$2: Q4.C, R36.2
- net 0V: now also Q2.E, Q4.E; no longer Q2.C, Q4.C
Other:
- moved on the sheet: Q2, Q4
Changed lines of the file:
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@@
 <?xml version="1.0" encoding="utf-8"?>
 <!DOCTYPE eagle SYSTEM "eagle.dtd">
-<eagle version="7.2.0">
+<eagle version="7.5.0">
 <drawing>
 <settings>
@@
 <instance part="CVOFFS-A" gate="G$1" x="35.56" y="111.76" rot="R90"/>
 <instance part="BIAS-A" gate="G$1" x="43.18" y="15.24"/>
-<instance part="Q2" gate="G$1" x="60.96" y="71.12"/>
+<instance part="Q2" gate="G$1" x="60.96" y="71.12" rot="MR180"/>
 <instance part="Q1" gate="G$1" x="50.8" y="86.36"/>
 <instance part="IC1" gate="A" x="30.48" y="86.36" rot="MR180"/>
@@
 <instance part="CVOFFS-B" gate="G$1" x="170.18" y="111.76" rot="R90"/>
 <instance part="BIAS-B" gate="G$1" x="177.8" y="15.24"/>
-<instance part="Q4" gate="G$1" x="195.58" y="71.12"/>
+<instance part="Q4" gate="G$1" x="195.58" y="71.12" rot="MR180"/>
 <instance part="Q3" gate="G$1" x="185.42" y="86.36"/>
 <instance part="R26" gate="G$1" x="149.86" y="73.66" rot="R90"/>
@@
 </segment>
 <segment>
-<pinref part="Q2" gate="G$1" pin="C"/>
-<wire x1="63.5" y1="76.2" x2="63.5" y2="78.74" width="0.1524" layer="91"/>
-<wire x1="63.5" y1="78.74" x2="71.12" y2="78.74" width="0.1524" layer="91"/>
 <pinref part="GND9" gate="1" pin="0V"/>
 <wire x1="71.12" y1="78.74" x2="71.12" y2="76.2" width="0.1524" layer="91"/>
+<wire x1="71.12" y1="78.74" x2="63.5" y2="78.74" width="0.1524" layer="91"/>
+<pinref part="Q2" gate="G$1" pin="E"/>
+<wire x1="63.5" y1="78.74" x2="63.5" y2="76.2" width="0.1524" layer="91"/>
 </segment>
 <segment>
@@
 </segment>
 <segment>
-<pinref part="Q4" gate="G$1" pin="C"/>
+<pinref part="GND20" gate="1" pin="0V"/>
+<wire x1="205.74" y1="78.74" x2="205.74" y2="76.2" width="0.1524" layer="91"/>
+<pinref part="Q4" gate="G$1" pin="E"/>
 <wire x1="198.12" y1="76.2" x2="198.12" y2="78.74" width="0.1524" layer="91"/>
 <wire x1="198.12" y1="78.74" x2="205.74" y2="78.74" width="0.1524" layer="91"/>
-<pinref part="GND20" gate="1" pin="0V"/>
-<wire x1="205.74" y1="78.74" x2="205.74" y2="76.2" width="0.1524" layer="91"/>
 </segment>
 <segment>
@@
 <pinref part="R11" gate="G$1" pin="2"/>
 <wire x1="53.34" y1="81.28" x2="53.34" y2="71.12" width="0.1524" layer="91"/>
-<wire x1="53.34" y1="68.58" x2="53.34" y2="71.12" width="0.1524" layer="91"/>
 <pinref part="Q2" gate="G$1" pin="B"/>
+<wire x1="53.34" y1="71.12" x2="53.34" y2="68.58" width="0.1524" layer="91"/>
 <wire x1="53.34" y1="71.12" x2="55.88" y2="71.12" width="0.1524" layer="91"/>
 <junction x="53.34" y="71.12"/>
-</segment>
-</net>
-<net name="N$9" class="0">
-<segment>
-<pinref part="Q2" gate="G$1" pin="E"/>
-<pinref part="R13" gate="G$1" pin="2"/>
 </segment>
 </net>
@@
 <pinref part="R34" gate="G$1" pin="2"/>
 <wire x1="187.96" y1="81.28" x2="187.96" y2="71.12" width="0.1524" layer="91"/>
-<wire x1="187.96" y1="68.58" x2="187.96" y2="71.12" width="0.1524" layer="91"/>
 <pinref part="Q4" gate="G$1" pin="B"/>
-<wire x1="187.96" y1="71.12" x2="190.5" y2="71.12" width="0.1524" layer="91"/>
+<wire x1="187.96" y1="71.12" x2="187.96" y2="68.58" width="0.1524" layer="91"/>
+<wire x1="190.5" y1="71.12" x2="187.96" y2="71.12" width="0.1524" layer="91"/>
 <junction x="187.96" y="71.12"/>
-</segment>
-</net>
-<net name="N$30" class="0">
-<segment>
-<pinref part="Q4" gate="G$1" pin="E"/>
-<pinref part="R36" gate="G$1" pin="2"/>
 </segment>
 </net>
@@
 </segment>
 </net>
+<net name="N$1" class="0">
+<segment>
+<pinref part="R13" gate="G$1" pin="2"/>
+<pinref part="Q2" gate="G$1" pin="C"/>
+</segment>
+</net>
+<net name="N$2" class="0">
+<segment>
+<pinref part="R36" gate="G$1" pin="2"/>
+<pinref part="Q4" gate="G$1" pin="C"/>
+</segment>
+</net>
