File: v2.0/schematics/eagle/quad.vca/quad.vca.main.brd (EAGLE design)
At the start: 100 x 80 mm, 66 parts, among them IC1 TL084P, IC2 LM13700N, J1 CV2-A, J2 CV1-A, J3 IN-A, J4 OUT-A, J5 CV2-B, J6 CV1-B, J7 IN-B, J8 OUT-B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

Commit message: Replaced trim pots with tested fixed values. Corrected error in PNP transisitor connection
Connections:
- net 0V: now also Q2.1, Q4.1; no longer Q2.3, Q4.3
- net N$30: now also Q4.3; no longer Q4.1
- net N$9: now also Q2.3; no longer Q2.1
Changed lines of the file:
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@@
 <?xml version="1.0" encoding="utf-8"?>
 <!DOCTYPE eagle SYSTEM "eagle.dtd">
-<eagle version="7.2.0">
+<eagle version="7.5.0">
 <drawing>
 <settings>
@@
 <contactref element="J4" pad="P$1"/>
 <contactref element="R4" pad="1"/>
-<contactref element="Q2" pad="3"/>
 <contactref element="R7" pad="1"/>
 <contactref element="IC2" pad="4"/>
@@
 <contactref element="J8" pad="P$1"/>
 <contactref element="R27" pad="1"/>
-<contactref element="Q4" pad="3"/>
 <contactref element="R30" pad="1"/>
 <contactref element="R38" pad="1"/>
@@
 <contactref element="R41" pad="1"/>
 <contactref element="IC2" pad="13"/>
+<contactref element="Q2" pad="1"/>
+<contactref element="Q4" pad="1"/>
 <wire x1="-33.02" y1="-201.93" x2="-33.02" y2="-218.44" width="0" layer="19" extent="1-1"/>
 <wire x1="-23.58" y1="-203.64" x2="-33.02" y2="-201.93" width="0" layer="19" extent="1-1"/>
@@
 <wire x1="-45.72" y1="-247.65" x2="-27.94" y2="-238.76" width="0" layer="19" extent="1-1"/>
 <wire x1="-45.72" y1="-252.73" x2="-45.72" y2="-247.65" width="0" layer="19" extent="1-1"/>
-<wire x1="2.54" y1="-227.33" x2="0" y2="-201.93" width="0" layer="19" extent="1-1"/>
-<wire x1="-5.08" y1="-252.73" x2="2.54" y2="-227.33" width="0" layer="19" extent="1-1"/>
+<wire x1="-2.54" y1="-227.33" x2="0" y2="-201.93" width="0" layer="19" extent="1-1"/>
+<wire x1="-5.08" y1="-252.73" x2="-2.54" y2="-227.33" width="0" layer="19" extent="1-1"/>
 <wire x1="-5.08" y1="-257.81" x2="-5.08" y2="-252.73" width="0" layer="19" extent="1-1"/>
 <wire x1="-45.72" y1="-160.02" x2="-33.02" y2="-201.93" width="0" layer="19" extent="1-1"/>
@@
 <wire x1="-35.56" y1="-41.91" x2="-45.72" y2="-53.34" width="0" layer="19" extent="1-1"/>
 <wire x1="-35.56" y1="-34.29" x2="-35.56" y2="-41.91" width="0" layer="19" extent="1-1"/>
-<wire x1="-31.75" y1="-13.97" x2="-35.56" y2="-34.29" width="0" layer="19" extent="1-1"/>
-<wire x1="-16.51" y1="3.81" x2="-31.75" y2="-13.97" width="0" layer="19" extent="1-1"/>
+<wire x1="-36.83" y1="-13.97" x2="-35.56" y2="-34.29" width="0" layer="19" extent="1-1"/>
+<wire x1="-16.51" y1="3.81" x2="-36.83" y2="-13.97" width="0" layer="19" extent="1-1"/>
 <wire x1="-23.58" y1="18.61" x2="-16.51" y2="3.81" width="0" layer="19" extent="1-1"/>
 <wire x1="-16.51" y1="20.32" x2="-23.58" y2="18.61" width="0" layer="19" extent="1-1"/>
@@
 <wire x1="-45.72" y1="-13.97" x2="-34.29" y2="-13.97" width="0" layer="19" extent="1-1"/>
 </signal>
-<signal name="N$9">
-<contactref element="Q2" pad="1"/>
-<contactref element="R13" pad="2"/>
-<wire x1="-36.83" y1="-13.97" x2="-38.1" y2="-73.66" width="0" layer="19" extent="1-1"/>
-</signal>
 <signal name="N$8">
 <contactref element="FEED-A" pad="A"/>
@@
 <wire x1="-45.72" y1="-240.03" x2="-7.62" y2="-247.65" width="0" layer="19" extent="1-1"/>
 </signal>
-<signal name="N$30">
-<contactref element="Q4" pad="1"/>
-<contactref element="R36" pad="2"/>
-<wire x1="-2.54" y1="-227.33" x2="2.54" y2="-247.65" width="0" layer="19" extent="1-1"/>
-</signal>
 <signal name="N$31">
 <contactref element="FEED-B" pad="A"/>
@@
 <wire x1="-16.51" y1="-238.76" x2="-43.18" y2="-34.29" width="0" layer="19" extent="1-1"/>
 </signal>
+<signal name="N$9">
+<contactref element="R13" pad="2"/>
+<contactref element="Q2" pad="3"/>
+<wire x1="-31.75" y1="-13.97" x2="-38.1" y2="-73.66" width="0" layer="19" extent="1-1"/>
+</signal>
+<signal name="N$30">
+<contactref element="R36" pad="2"/>
+<contactref element="Q4" pad="3"/>
+<wire x1="2.54" y1="-227.33" x2="2.54" y2="-247.65" width="0" layer="19" extent="1-1"/>
+</signal>
 </signals>
