File: v2.0/schematics/eagle/quad.vca/quad.exp.vca.pnl.brd (EAGLE design)
At the start: 100 x 80 mm, 66 parts, among them IC1 TL084P, IC2 LM13700N, J1 CV2-A, J2 CV1-A, J3 IN-A, J4 OUT-A, J5 CV2-B, J6 CV1-B, J7 IN-B, J8 OUT-B, Q1 2N3904, Q2 2N3906, Q3 2N3904, Q4 2N3906

Commit message: Split quad.exp.vca into main and pnl boards with completed autorouting
Parts:
- removed BIAS-A, BIAS-B: 100K, pot:PT-10S
- removed CV2ATT-A, CV2ATT-B, CVOFFS-A, CVOFFS-B: 100K, _common:R-VAR
- removed FEED-A, FEED-B: 2K, pot:PT-10S
- removed IC1: TL084P, linear:DIL14
- removed IC2: LM13700N, ota:DIL16
- removed Q1, Q3: 2N3904, _common:TO92
- removed Q2, Q4: 2N3906, _common:TO92
- removed R11: 120K, resistor:0207/7
- removed R12: 2.2M, resistor:0207/7
- removed R14, R37: 470K, resistor:0207/7
- removed R15, R38: 47K, resistor:0207/7
- removed R17, R2, R21, R24, R25, R26, R3, R40, R44, R8: 100K, resistor:0207/7
- removed R18, R41: 470, resistor:0207/7
- removed R22, R45: 30K, resistor:0207/7
- removed R23, R36: 20K, resistor:0207/7
- removed R27, R32, R39, R9: 2K, resistor:0207/7
- removed R30, R7: 150, resistor:0207/7
- removed R42: 4.7K, resistor:0207/7
- added J10: CV4, jacks:ACJM-MV35-2S
- added J11: IN4, jacks:ACJM-MV35-2S
- added J12: OUT4, jacks:ACJM-MV35-2S
- added J9: OUT3, jacks:ACJM-MV35-2S
- added R49: 100K, resistor:0207/7
- added R50, R58: 1K, resistor:0207/7
- J1: value CV2-A -> CV1
- J2: value CV1-A -> IN1
- J3: value IN-A -> OUT1
- J4: value OUT-A -> CV2
- J5: value CV2-B -> IN2
- J6: value CV1-B -> OUT2
- J7: value IN-B -> CV3
- J8: value OUT-B -> IN3
- JP1: value LOG/LIN -> VCA1-2; device pinhead:1X03 -> pinhead:1X10
- JP2: value LOG/LIN -> VCA3-4; device pinhead:1X03 -> pinhead:1X10
- R13: value 20K -> 1K
- R16, R4: value 2K -> 100K
- R19: value 4.7K -> 100K
- R28, R5: value 100K -> 1K
- R34: value 120K -> 100K
- R35: value 2.2M -> 1K
- R46: value 20K -> 100K
- moved R46 312.4 mm to (72.4, 38.1), turned to 180 degrees
- moved R43 308.6 mm to (55.9, 38.1), turned to 180 degrees
- moved R28 299.1 mm to (38.1, 38.1)
- moved JP2 280.3 mm to (92.1, 19.7), flipped to the bottom, turned to 90 degrees
- moved R31 270.8 mm to (74.9, 1.27), turned to 180 degrees
- moved R35 268.3 mm to (64.8, 1.27), turned to 180 degrees
- moved R34 257.5 mm to (54.6, 1.27)
- moved J6 239.4 mm to (45.7, 24.1)
- moved J5 238.2 mm to (45.7, 6.35)
- moved J7 229.0 mm to (78.7, 6.35)
- moved J8 217.4 mm to (62.2, 6.35)
- moved R16 213.3 mm to (22.9, 38.1), turned to 180 degrees
- moved JP1 211.5 mm to (9.53, 19.7), flipped to the bottom, turned to 90 degrees
- moved R1 164.9 mm to (24.1, 1.27), turned to 180 degrees
- moved J1 161.1 mm to (29.2, 6.35)
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Connections:
- removed net +12V: BIAS-A.E, BIAS-B.E, CVOFFS-A.R2, CVOFFS-B.R2, IC1.4, IC2.11, Q1.3, Q3.3, R14.2, R17.2, R26.2, R3.2, R37.2, R40.2
- removed net -12V: BIAS-A.A, BIAS-B.A, CVOFFS-A.R1, CVOFFS-B.R1, IC1.11, IC2.6, R11.1, R19.1, R23.1, R34.1, R42.1, R46.1
- removed net N$10: JP1.1, R13.1
- removed net N$11: J3.P$3, R5.1
- removed net N$12: FEED-A.E, FEED-A.S, IC2.3, R5.2
- removed net N$13: IC2.8, R19.2, R20.1
- removed net N$14: BIAS-A.S, R12.1
- removed net N$15: IC2.5, IC2.7, R12.2, R14.1, R15.2
- removed net N$17: CV2ATT-A.VAR, R1.2
- removed net N$18: JP1.3, R22.1, R23.2
- removed net N$19: IC1.5, R17.1, R18.2
- removed net N$20: IC1.6, R16.2, R21.1
- removed net N$21: IC2.1, JP1.2
- removed net N$22: IC1.7, R21.2, R22.2
- removed net N$23: J6.P$2, J6.P$3, R25.1
- removed net N$25: IC1.10, R26.1, R27.2
- removed net N$26: IC1.9, R24.1, R25.2, R31.2, R32.1
- removed net N$27: CVOFFS-B.VAR, R31.1
- removed net N$28: IC1.8, Q3.2, R32.2, R39.1
- removed net N$29: Q3.1, Q4.2, R34.2
- removed net N$30: Q4.3, R36.2
- removed net N$32: J7.P$3, R28.1
- removed net N$33: FEED-B.E, FEED-B.S, IC2.14, R28.2
- removed net N$34: BIAS-B.S, R35.1
- removed net N$35: IC2.10, IC2.12, R35.2, R37.1, R38.2
- removed net N$36: IC2.9, R42.2, R43.1
- removed net N$37: CV2ATT-B.R2, J5.P$2, J5.P$3
- removed net N$38: CV2ATT-B.VAR, R24.2
- removed net N$39: IC1.12, R40.1, R41.2
- removed net N$40: IC1.13, R39.2, R44.1
- removed net N$41: IC1.14, R44.2, R45.2
- removed net N$43: JP2.3, R45.1, R46.2
- removed net N$44: IC2.16, JP2.2
- removed net N$9: Q2.3, R13.2
- new net CV1: JP1.5, R1.1
- new net CV2: JP1.6, R16.1
- new net CV3: JP2.5, R31.1
- new net CV4: JP2.6, R46.1
- new net IN1: JP1.3, R4.2, R5.2
- new net IN2: JP1.7, R19.2, R20.2
- new net IN3: JP2.3, R34.2, R35.2
- new net IN4: JP2.7, R49.2, R50.2
- new net OUT1: JP1.4, R13.1
- new net OUT2: JP1.8, R28.1
- new net OUT3: JP2.4, R43.1
- new net OUT4: JP2.8, R58.1
- net 0V: now also J10.P$1, J11.P$1, J12.P$1, J2.P$2, J9.P$1, JP1.1, JP1.10, JP1.2, JP1.9, JP2.1, JP2.10, JP2.2, JP2.9, R20.1, R35.1, R5.1, R50.1; no longer CV2ATT-A.R1, CV2ATT-B.R1, IC2.13, IC2.4, J3.P$2, J7.P$2, Q2.1, Q4.1, R15.1, R18.1, R27.1, R30.1, R38.1, R4.1, R41.1, R7.1
- net N$1: now also J9.P$2, J9.P$3, R43.2; no longer J2.P$2, J2.P$3, R2.1
- net N$16: now also J4.P$2, R1.2; no longer CV2ATT-A.R2
- net N$2: now also J3.P$2, J3.P$3, R13.2; no longer J4.P$2, J4.P$3, R20.2
- net N$24: now also J6.P$2, J6.P$3, R28.2; no longer J8.P$2, J8.P$3, R43.2
- net N$3: now also J2.P$3, J5.P$2, R4.1; no longer IC1.3, R3.1, R4.2
- net N$31: now also J12.P$2, J12.P$3, R58.2; no longer FEED-B.A, R30.2
- net N$4: now also J5.P$3, J8.P$2, R19.1; no longer IC1.2, R1.1, R2.2, R8.2, R9.1
- net N$42: now also J11.P$3, R49.1; no longer JP2.1, R36.1
- net N$5: now also J11.P$2, J8.P$3, R34.1; no longer CVOFFS-A.VAR, R8.1
- net N$6: now also J10.P$3, R46.2; no longer IC1.1, Q1.2, R16.1, R9.2
- net N$7: now also J10.P$2, J7.P$3, R31.2; no longer Q1.1, Q2.2, R11.2
- net N$8: now also J4.P$3, J7.P$2, R16.2; no longer FEED-A.A, R7.2
Routing:
- net 0V: track 0.00 -> 248.7 mm
- net N$8: track 0.00 -> 109.0 mm
- net N$5: track 0.00 -> 61.0 mm, vias 0 -> 1
- net N$3: track 0.00 -> 57.5 mm, vias 0 -> 1
- net OUT2: track 0.00 -> 54.5 mm
- net N$4: track 0.00 -> 46.9 mm
- net OUT3: track 0.00 -> 45.7 mm
- net IN3: track 0.00 -> 44.0 mm
- net IN2: track 0.00 -> 41.9 mm, vias 0 -> 1
- net CV1: track 0.00 -> 40.8 mm
- net CV3: track 0.00 -> 35.7 mm
- net IN4: track 0.00 -> 28.9 mm
- net CV2: track 0.00 -> 28.0 mm, vias 0 -> 1
- net CV4: track 0.00 -> 27.0 mm
- net N$16: track 0.00 -> 25.3 mm
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Other:
- board size 100 x 80 mm -> 98.7 x 39.4 mm
- board text added: "dlp.quad.exp.vca.pnl v2.0.0.rev1"
