File: v2.0/schematics/eagle/digtal.noise.gen/digital.noise.gen.sch (EAGLE design)
At the start: 15 parts, among them IC1 TL072P

Commit message: Added scaled digial noise out and tune input on PIC
Parts:
- added J1: DIG NOISE OUT, jacks:ACJM-MV35-2S
- added RV2: NOISE TUNE, _common:R-VAR
- R2: value ?? -> 1M; device _common:R-US_0207/7 -> resistor:R-TRIMM3339P
- R3: value ?? -> 1K
- R4: value ?? -> 220K
Connections:
- new net N$6: J1.P$2, R3.1
- new net N$8: RV2.P$1, U$1.RA0/AN0
- net +12V: now also R2.E; no longer R2.2
- net +5V: now also RV2.2
- net -12V: now also R2.A; no longer R3.1
- net 0V: now also J1.P$1, RV2.1
- net N$15: now also R2.S; no longer R2.1, R3.2
- net N$16: now also R3.2
Other:
- note added: "Inveting Ref: http://electronics.stackexchange.com/questions/37095/level-shifting-a-2-5v-signal-to-0-5v Trim split is 382K to +12V and 511K to -12V This generates about +5.5V/-5.5V from a +5V/0V wave"
- note removed: "Inveting Ref: http://electronics.stackexchange.com/questions/37095/level-shifting-a-2-5v-signal-to-0-5v"
- moved on the sheet: C1, D1, R1, R3, R5
Changed lines of the file:
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@@
 <part name="P+5" library="supply1" deviceset="+5V" device=""/>
 <part name="IC1" library="_common" deviceset="TL072" device="P"/>
-<part name="R3" library="_common" deviceset="R-US_" device="0207/7" value="??"/>
-<part name="R4" library="_common" deviceset="R-US_" device="0207/7" value="??"/>
+<part name="R4" library="_common" deviceset="R-US_" device="0207/7" value="220K"/>
 <part name="R5" library="_common" deviceset="R-US_" device="0207/7" value="100K"/>
 <part name="P-3" library="supply1" deviceset="-12V" device=""/>
@@
 <part name="P+7" library="supply1" deviceset="+12V" device=""/>
 <part name="P-2" library="supply1" deviceset="-12V" device=""/>
-<part name="R2" library="_common" deviceset="R-US_" device="0207/7" value="??"/>
+<part name="R2" library="resistor" deviceset="R-TRIMM" device="3339P" value="1M"/>
+<part name="R3" library="_common" deviceset="R-US_" device="0207/7" value="1K"/>
+<part name="J1" library="jacks" deviceset="ACJM-MV35-2S" device="" value="DIG NOISE OUT"/>
+<part name="GND7" library="supply1" deviceset="0V" device=""/>
+<part name="P+8" library="supply1" deviceset="+5V" device=""/>
+<part name="GND8" library="supply1" deviceset="0V" device=""/>
+<part name="RV2" library="_common" deviceset="R-VAR" device="" value="NOISE TUNE"/>
 </parts>
 <sheets>
 <sheet>
 <plain>
-<text x="134.62" y="50.8" size="1.778" layer="91">Inveting
-Ref: http://electronics.stackexchange.com/questions/37095/level-shifting-a-2-5v-signal-to-0-5v</text>
+<text x="116.84" y="76.2" size="1.778" layer="91">Inveting
+Ref: http://electronics.stackexchange.com/questions/37095/level-shifting-a-2-5v-signal-to-0-5v
+Trim split is 382K to +12V and 511K to -12V
+This generates about +5.5V/-5.5V from a +5V/0V wave</text>
 </plain>
 <instances>
@@
 <instance part="GND1" gate="1" x="55.88" y="10.16"/>
 <instance part="P-1" gate="1" x="66.04" y="76.2"/>
-<instance part="P+2" gate="1" x="2.54" y="40.64"/>
-<instance part="C1" gate="G$1" x="2.54" y="10.16"/>
-<instance part="R1" gate="G$1" x="2.54" y="25.4" rot="R90"/>
-<instance part="D1" gate="G$1" x="2.54" y="33.02" rot="R270"/>
+<instance part="P+2" gate="1" x="0" y="40.64"/>
+<instance part="C1" gate="G$1" x="0" y="10.16"/>
+<instance part="R1" gate="G$1" x="0" y="25.4" rot="R90"/>
+<instance part="D1" gate="G$1" x="0" y="33.02" rot="R270"/>
 <instance part="JP1" gate="A" x="53.34" y="25.4" rot="R90"/>
 <instance part="JP2" gate="A" x="53.34" y="88.9" rot="R180"/>
 <instance part="Q1" gate="G$1" x="111.76" y="40.64"/>
-<instance part="GND2" gate="1" x="2.54" y="2.54"/>
+<instance part="GND2" gate="1" x="0" y="2.54"/>
 <instance part="P+3" gate="1" x="10.16" y="71.12"/>
 <instance part="GND3" gate="1" x="10.16" y="33.02"/>
@@
 <instance part="P+5" gate="1" x="40.64" y="99.06"/>
 <instance part="IC1" gate="A" x="134.62" y="60.96" rot="MR180"/>
-<instance part="R3" gate="G$1" x="121.92" y="53.34" rot="R90"/>
 <instance part="R4" gate="G$1" x="134.62" y="71.12" rot="R180"/>
-<instance part="R5" gate="G$1" x="104.14" y="63.5" rot="R180"/>
-<instance part="IC1" gate="P" x="81.28" y="88.9"/>
-<instance part="P-3" gate="1" x="81.28" y="78.74"/>
-<instance part="P+6" gate="1" x="81.28" y="99.06"/>
-<instance part="P+7" gate="1" x="121.92" y="78.74"/>
-<instance part="P-2" gate="1" x="121.92" y="45.72"/>
-<instance part="R2" gate="G$1" x="121.92" y="71.12" rot="R90"/>
+<instance part="R5" gate="G$1" x="109.22" y="63.5" rot="R180"/>
+<instance part="IC1" gate="P" x="76.2" y="86.36"/>
+<instance part="P-3" gate="1" x="76.2" y="76.2"/>
+<instance part="P+6" gate="1" x="76.2" y="96.52"/>
+<instance part="P+7" gate="1" x="119.38" y="60.96"/>
+<instance part="P-2" gate="1" x="119.38" y="45.72"/>
+<instance part="R2" gate="G$1" x="119.38" y="53.34"/>
+<instance part="R3" gate="G$1" x="162.56" y="60.96" rot="R180"/>
+<instance part="J1" gate="G$1" x="182.88" y="53.34" rot="MR0"/>
+<instance part="GND7" gate="1" x="182.88" y="50.8"/>
+<instance part="P+8" gate="1" x="0" y="71.12"/>
+<instance part="GND8" gate="1" x="0" y="50.8"/>
+<instance part="RV2" gate="G$1" x="0" y="60.96" rot="MR90"/>
 </instances>
 <busses>
@@
 <segment>
 <pinref part="U$1" gate="A" pin="RA5/~MCLR/VPP"/>
-<wire x1="10.16" y1="48.26" x2="7.62" y2="48.26" width="0.1524" layer="91"/>
-<wire x1="7.62" y1="48.26" x2="7.62" y2="17.78" width="0.1524" layer="91"/>
+<wire x1="10.16" y1="48.26" x2="5.08" y2="48.26" width="0.1524" layer="91"/>
+<wire x1="5.08" y1="48.26" x2="5.08" y2="17.78" width="0.1524" layer="91"/>
 <pinref part="JP1" gate="A" pin="1"/>
-<wire x1="7.62" y1="17.78" x2="48.26" y2="17.78" width="0.1524" layer="91"/>
+<wire x1="5.08" y1="17.78" x2="48.26" y2="17.78" width="0.1524" layer="91"/>
 <wire x1="48.26" y1="17.78" x2="48.26" y2="22.86" width="0.1524" layer="91"/>
-<wire x1="7.62" y1="17.78" x2="2.54" y2="17.78" width="0.1524" layer="91"/>
-<junction x="7.62" y="17.78"/>
+<wire x1="5.08" y1="17.78" x2="0" y2="17.78" width="0.1524" layer="91"/>
+<junction x="5.08" y="17.78"/>
 <pinref part="C1" gate="G$1" pin="1"/>
-<wire x1="2.54" y1="17.78" x2="2.54" y2="15.24" width="0.1524" layer="91"/>
+<wire x1="0" y1="17.78" x2="0" y2="15.24" width="0.1524" layer="91"/>
 <pinref part="R1" gate="G$1" pin="1"/>
-<wire x1="2.54" y1="17.78" x2="2.54" y2="20.32" width="0.1524" layer="91"/>
-<junction x="2.54" y="17.78"/>
+<wire x1="0" y1="17.78" x2="0" y2="20.32" width="0.1524" layer="91"/>
+<junction x="0" y="17.78"/>
 </segment>
 </net>
@@
 <junction x="48.26" y="83.82"/>
 </segment>
+<segment>
+<pinref part="J1" gate="G$1" pin="P$1"/>
+<pinref part="GND7" gate="1" pin="0V"/>
+</segment>
+<segment>
+<pinref part="GND8" gate="1" pin="0V"/>
+<pinref part="RV2" gate="G$1" pin="1"/>
+<wire x1="0" y1="53.34" x2="0" y2="55.88" width="0.1524" layer="91"/>
+</segment>
 </net>
 <net name="+5V" class="0">
@@
 <pinref part="D1" gate="G$1" pin="A"/>
 <pinref part="P+2" gate="1" pin="+5V"/>
-<wire x1="2.54" y1="35.56" x2="2.54" y2="38.1" width="0.1524" layer="91"/>
+<wire x1="0" y1="35.56" x2="0" y2="38.1" width="0.1524" layer="91"/>
 </segment>
 <segment>
@@
 <pinref part="P+5" gate="1" pin="+5V"/>
 <wire x1="40.64" y1="93.98" x2="40.64" y2="96.52" width="0.1524" layer="91"/>
+</segment>
+<segment>
+<pinref part="RV2" gate="G$1" pin="2"/>
+<pinref part="P+8" gate="1" pin="+5V"/>
+<wire x1="0" y1="68.58" x2="0" y2="66.04" width="0.1524" layer="91"/>
 </segment>
 </net>
@@
 </segment>
 <segment>
-<pinref part="R3" gate="G$1" pin="1"/>
+<pinref part="R2" gate="G$1" pin="A"/>
 <pinref part="P-2" gate="1" pin="-12V"/>
 </segment>
@@
 </segment>
 <segment>
+<pinref part="R2" gate="G$1" pin="E"/>
 <pinref part="P+7" gate="1" pin="+12V"/>
-<pinref part="R2" gate="G$1" pin="2"/>
 </segment>
 </net>
@@
 <pinref part="U$1" gate="A" pin="RB1/SDI/SDA"/>
 <pinref part="R5" gate="G$1" pin="2"/>
-<wire x1="96.52" y1="63.5" x2="99.06" y2="63.5" width="0.1524" layer="91"/>
+<wire x1="96.52" y1="63.5" x2="104.14" y2="63.5" width="0.1524" layer="91"/>
 </segment>
 </net>
@@
 <pinref part="R5" gate="G$1" pin="1"/>
 <pinref part="IC1" gate="A" pin="-IN"/>
-<wire x1="109.22" y1="63.5" x2="124.46" y2="63.5" width="0.1524" layer="91"/>
+<wire x1="114.3" y1="63.5" x2="124.46" y2="63.5" width="0.1524" layer="91"/>
 <wire x1="124.46" y1="63.5" x2="127" y2="63.5" width="0.1524" layer="91"/>
 <pinref part="R4" gate="G$1" pin="2"/>
@@
 <net name="N$15" class="0">
 <segment>
-<pinref part="R3" gate="G$1" pin="2"/>
 <pinref part="IC1" gate="A" pin="+IN"/>
-<wire x1="121.92" y1="58.42" x2="127" y2="58.42" width="0.1524" layer="91"/>
-<pinref part="R2" gate="G$1" pin="1"/>
-<wire x1="121.92" y1="66.04" x2="121.92" y2="58.42" width="0.1524" layer="91"/>
-<junction x="121.92" y="58.42"/>
+<wire x1="124.46" y1="58.42" x2="127" y2="58.42" width="0.1524" layer="91"/>
+<pinref part="R2" gate="G$1" pin="S"/>
+<wire x1="124.46" y1="58.42" x2="124.46" y2="53.34" width="0.1524" layer="91"/>
 </segment>
 </net>
@@
 <wire x1="147.32" y1="60.96" x2="157.48" y2="60.96" width="0.1524" layer="91"/>
 <junction x="147.32" y="60.96"/>
-</segment>
-</net>
+<pinref part="R3" gate="G$1" pin="2"/>
+</segment>
+</net>
+<net name="N$6" class="0">
+<segment>
+<pinref part="R3" gate="G$1" pin="1"/>
+<pinref part="J1" gate="G$1" pin="P$2"/>
+</segment>
+</net>
+<net name="N$8" class="0">
+<segment>
+<pinref part="RV2" gate="G$1" pin="P$1"/>
+<pinref part="U$1" gate="A" pin="RA0/AN0"/>
+<wire x1="5.08" y1="60.96" x2="10.16" y2="60.96" width="0.1524" layer="91"/>
+</segment>
+</net>
