File: v2.0/schematics/eagle/vcf.lp.4p.24db/vcf.lp.4p.24db-rev1.brd (EAGLE design)
At the start: 98.7 x 54.6 mm, 83 parts, among them IC1 TL082P, IC2 TL084P, IC3 TL084P, IC4 LM13700N, IC5 LM13700N, J1 IN, J2 OUT, T1 2N3904, T2 2N3904, T3 2N3906, T4 2N3906, T5 2N3906, T6 2N3906

Commit message: Panel revisions; VCF-LP board layout
Parts:
- moved RV3 643.6 mm to (66.0, 67.3), turned to 180 degrees
- moved R4 628.2 mm to (83.8, 55.9), turned to 270 degrees
- moved IC2 627.8 mm to (49.5, 44.5)
- moved R43 609.7 mm to (61.0, 47.0), turned to 90 degrees
- moved R42 609.1 mm to (50.8, 53.3)
- moved JP3 604.9 mm to (40.6, 58.4)
- moved C12 546.7 mm to (48.3, 50.8)
- moved C11 525.8 mm to (49.5, 36.8), turned to 270 degrees
- moved C9 520.9 mm to (85.1, 38.1), turned to 90 degrees
- moved RV2 515.8 mm to (43.2, 67.3), turned to 180 degrees
- moved C10 513.6 mm to (85.1, 22.9), turned to 90 degrees
- moved C8 502.4 mm to (44.5, 36.8), turned to 270 degrees
- moved C7 480.1 mm to (44.5, 21.6), turned to 270 degrees
- moved R25 376.1 mm to (20.3, 39.4), turned to 90 degrees
- moved R27 374.1 mm to (58.4, 38.1)
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Connections:
- removed net V+: IC4.11, IC5.11
- removed net V-: IC4.6, IC5.6
- net +12V: now also IC4.11, IC5.11
- net -12V: now also IC4.6, IC5.6
Routing:
- net +12V: track 59.0 -> 261.7 mm
- net N$14: track 0.00 -> 153.3 mm
- net -12V: track 198.0 -> 278.8 mm, vias 3 -> 0
- net N$47: track 0.00 -> 73.0 mm
- net N$39: track 0.00 -> 60.9 mm
- net N$5: track 0.00 -> 59.8 mm
- net N$44: track 0.00 -> 58.5 mm
- net N$41: track 0.00 -> 49.6 mm
- net N$7: track 0.00 -> 46.9 mm
- net N$27: track 0.00 -> 46.9 mm
- net N$30: track 0.00 -> 46.2 mm
- net N$25: track 0.00 -> 43.4 mm
- net N$26: track 0.00 -> 43.4 mm
- net N$50: track 0.00 -> 37.8 mm
- net N$17: track 0.00 -> 36.8 mm
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Other:
- board size 98.7 x 54.6 mm -> 98.7 x 71.1 mm
- board text added: "CUT INIT"
- board text added: "CUTOFF"
- board text added: "CV ATT"
- board text added: "IN"
- board text added: "OUT"
- board text added: "RES"
- board text added: "VCF-LP rev1"
- board text removed: "ATTEN"
- board text removed: "BIAS"
- board text removed: "CV IN"
- board text removed: "CV INIT"
- board text removed: "LFOVCA rev2"
- board text removed: "MIN LVL"
- board text removed: "OFFSET"
- board text removed: "RATE"
- board text removed: "ROUND"
- board text removed: "SINE"
- board text removed: "SYMM"

Commit message: VCF-LP: Update names; cam export
Parts:
- moved JP2 18.0 mm to (14.0, 55.9), turned to 0 degrees
Routing:
- net N$3: track 13.8 -> 38.8 mm
Other:
- board text added: "+"
- board text added: "-"
- board text added: "CV IN"
- board text added: "RES BOOST"

Commit message: Updatd values for VCFLP
Parts:
- R8: value 1M -> 470K
Changed lines of the file:
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@@
 <attribute name="VALUE" x="58.9788" y="52.324" size="1.27" layer="27" ratio="10" rot="R90"/>
 </element>
-<element name="R8" library="resistor" package="0207/7" value="1M" x="29.21" y="50.8" smashed="yes" rot="R180">
+<element name="R8" library="resistor" package="0207/7" value="470K" x="29.21" y="50.8" smashed="yes" rot="R180">
 <attribute name="NAME" x="29.083" y="49.53" size="1.27" layer="25" ratio="10" rot="R180"/>
 <attribute name="VALUE" x="31.496" y="51.3588" size="1.27" layer="27" ratio="10" rot="R180"/>

Commit message: VCFLP: additional tweaks to values; added notes for trimmer and cuttoff trace issues
Parts:
- R25: value 20K -> 27K
- R43: value 100K -> 150K
Changed lines of the file:
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@@
 <attribute name="VALUE" x="56.134" y="37.5412" size="1.27" layer="27" ratio="10"/>
 </element>
-<element name="R25" library="resistor" package="0207/7" value="20K" x="20.32" y="39.37" smashed="yes" rot="R90">
+<element name="R25" library="resistor" package="0207/7" value="27K" x="20.32" y="39.37" smashed="yes" rot="R90">
 <attribute name="NAME" x="18.415" y="43.942" size="1.27" layer="25" ratio="10" rot="R90"/>
 <attribute name="VALUE" x="20.8788" y="37.084" size="1.27" layer="27" ratio="10" rot="R90"/>
@@
 <attribute name="VALUE" x="48.514" y="52.7812" size="1.27" layer="27" ratio="10"/>
 </element>
-<element name="R43" library="resistor" package="0207/7" value="100K" x="60.96" y="46.99" smashed="yes" rot="R90">
+<element name="R43" library="resistor" package="0207/7" value="150K" x="60.96" y="46.99" smashed="yes" rot="R90">
 <attribute name="NAME" x="63.754" y="44.45" size="1.27" layer="25" ratio="10" rot="R90"/>
 <attribute name="VALUE" x="61.5188" y="44.704" size="1.27" layer="27" ratio="10" rot="R90"/>
