File: v2.0/schematics/eagle/lfovca/lfovca-rev3.brd (EAGLE design)
At the start: 98.7 x 54.6 mm, 66 parts, among them IC1 TL082P, IC2 TL084P, T1 2N3904, T2 2N3904, T3 2N3904, T4 BC547, T5 BC547, T6 BC547

Commit message: Corrected R-VAR pin 2 & 3 mapping for VCFLP and LFOVCA
Connections:
- net +12V: now also RV3.3; no longer RV3.2
- net N$1: now also RV3.2; no longer RV3.3
- net N$13: now also RV1.3; no longer RV1.2
- net N$16: now also RV1.2; no longer RV1.3
- net N$24: now also RV2.3; no longer RV2.2
- net N$3: now also RV2.2; no longer RV2.3
Routing:
- net N$3: track 36.3 -> 43.4 mm, vias 0 -> 1
- net N$1: track 28.6 -> 35.0 mm
- net N$24: track 28.1 -> 23.8 mm
- net +12V: track 181.2 -> 183.3 mm
- net N$13: track 43.9 -> 42.4 mm
Other:
- board text added: "LFOVCA rev3"
- board text removed: "LFOVCA rev2"
- board text removed: "R-VAR PIN MAP IS WRONG! Pins 2 and 3 are swapped!!!"
Changed lines of the file:
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@@
 <wire x1="0" y1="54.6" x2="0" y2="0" width="0" layer="20"/>
 <wire x1="1.27" y1="1.27" x2="1.27" y2="6.35" width="0.254" layer="21"/>
-<text x="40.64" y="2.54" size="1.778" layer="25">LFOVCA rev2</text>
+<text x="40.64" y="2.54" size="1.778" layer="25">LFOVCA rev3</text>
 <text x="44.45" y="17.78" size="1.778" layer="25" align="center">BIAS</text>
 <text x="54.61" y="17.78" size="1.778" layer="25" align="center">SYMM</text>
@@
 <text x="30.48" y="43.815" size="1.778" layer="25" align="bottom-right">CV IN</text>
 <text x="12.7" y="43.815" size="1.778" layer="25" align="bottom-right">SINE</text>
-<text x="81.28" y="55.88" size="1.778" layer="51">R-VAR PIN MAP
-IS WRONG!
-Pins 2 and 3
-are swapped!!!</text>
-<text x="58.42" y="55.88" size="1.778" layer="51">R-VAR PIN MAP
-IS WRONG!
-Pins 2 and 3
-are swapped!!!</text>
-<text x="35.56" y="55.88" size="1.778" layer="51">R-VAR PIN MAP
-IS WRONG!
-Pins 2 and 3
-are swapped!!!</text>
 </plain>
 <attributes>
@@
 </signal>
 <signal name="N$1">
+<contactref element="RV3" pad="2"/>
+<contactref element="R16" pad="1"/>
+<wire x1="35.56" y1="43.18" x2="37.795196875" y2="45.415196875" width="0.4064" layer="1"/>
+<wire x1="37.795196875" y1="45.415196875" x2="53.392159375" y2="45.415196875" width="0.4064" layer="1"/>
+<wire x1="53.392159375" y1="45.415196875" x2="60.3771625" y2="52.4002" width="0.4064" layer="1"/>
+<wire x1="60.3771625" y1="52.4002" x2="64.4398" y2="52.4002" width="0.4064" layer="1"/>
+<wire x1="64.4398" y1="52.4002" x2="66.04" y2="50.8" width="0.4064" layer="1"/>
+</signal>
+<signal name="+12V" class="1">
 <contactref element="RV3" pad="3"/>
-<contactref element="R16" pad="1"/>
-<wire x1="40.64" y1="48.26" x2="35.56" y2="43.18" width="0.4064" layer="1"/>
-<wire x1="61.04" y1="50.8" x2="58.5" y2="48.26" width="0.4064" layer="1"/>
-<wire x1="58.5" y1="48.26" x2="40.64" y2="48.26" width="0.4064" layer="1"/>
-</signal>
-<signal name="+12V" class="1">
-<contactref element="RV3" pad="2"/>
 <contactref element="IC2" pad="4"/>
 <contactref element="IC1" pad="8"/>
@@
 <wire x1="43.5" y1="13" x2="37.8" y2="13" width="0.8128" layer="1"/>
 <wire x1="37.8" y1="13" x2="35.56" y2="15.24" width="0.8128" layer="1"/>
-<wire x1="66.04" y1="50.8" x2="69.85" y2="46.99" width="0.8128" layer="1"/>
-<wire x1="69.85" y1="46.99" x2="69.85" y2="35.56" width="0.8128" layer="1"/>
+<wire x1="61.04" y1="50.8" x2="69.85" y2="41.99" width="0.8128" layer="1"/>
+<wire x1="69.85" y1="41.99" x2="69.85" y2="36.322" width="0.8128" layer="1"/>
+<wire x1="69.85" y1="36.322" x2="69.85" y2="35.56" width="0.8128" layer="1"/>
 </signal>
 <signal name="-12V" class="1">
@@
 <contactref element="IC1" pad="7"/>
 <contactref element="C9" pad="1"/>
-<contactref element="RV1" pad="2"/>
-<wire x1="88.5" y1="36.5" x2="87.625" y2="35.625" width="0.4064" layer="1"/>
-<wire x1="87.625" y1="35.625" x2="86.5" y2="34.5" width="0.4064" layer="1"/>
-<wire x1="86.5" y1="34.5" x2="86.36" y2="34.29" width="0.4064" layer="1"/>
-<wire x1="88.9" y1="50.8" x2="88.5" y2="50.4" width="0.4064" layer="1"/>
-<wire x1="88.5" y1="50.4" x2="88.5" y2="36.5" width="0.4064" layer="1"/>
-<wire x1="91.44" y1="17.94" x2="91.44" y2="17.78" width="0.4064" layer="1"/>
-<wire x1="87.625" y1="35.625" x2="93.98" y2="29.27" width="0.4064" layer="1"/>
-<wire x1="93.98" y1="29.27" x2="93.98" y2="20.48" width="0.4064" layer="1"/>
-<wire x1="93.98" y1="20.48" x2="91.44" y2="17.94" width="0.4064" layer="1"/>
+<contactref element="RV1" pad="3"/>
 <wire x1="91.44" y1="17.78" x2="91.25" y2="17.59" width="0.4064" layer="1"/>
 <wire x1="91.25" y1="17.59" x2="91.25" y2="16.32" width="0.4064" layer="1"/>
 <wire x1="91.25" y1="16.32" x2="88.9" y2="13.97" width="0.4064" layer="1"/>
+<wire x1="86.36" y1="34.29" x2="87.648071875" y2="34.29" width="0.4064" layer="16"/>
+<wire x1="87.648071875" y1="34.29" x2="92.202" y2="29.736071875" width="0.4064" layer="16"/>
+<wire x1="92.202" y1="29.736071875" x2="92.202" y2="26.924" width="0.4064" layer="16"/>
+<wire x1="92.202" y1="26.924" x2="91.44" y2="26.162" width="0.4064" layer="16"/>
+<wire x1="91.44" y1="26.162" x2="91.44" y2="17.78" width="0.4064" layer="16"/>
+<wire x1="83.9" y1="50.8" x2="83.9" y2="36.75" width="0.4064" layer="1"/>
+<wire x1="83.9" y1="36.75" x2="86.36" y2="34.29" width="0.4064" layer="1"/>
 </signal>
 <signal name="N$16">
-<contactref element="RV1" pad="3"/>
+<contactref element="RV1" pad="2"/>
 <contactref element="R2" pad="1"/>
-<wire x1="84.5" y1="40" x2="86.36" y2="38.14" width="0.4064" layer="1"/>
-<wire x1="86.36" y1="38.14" x2="86.36" y2="38.1" width="0.4064" layer="1"/>
-<wire x1="83.9" y1="50.8" x2="84.5" y2="50.2" width="0.4064" layer="1"/>
-<wire x1="84.5" y1="50.2" x2="84.5" y2="40" width="0.4064" layer="1"/>
+<wire x1="88.9" y1="50.8" x2="88.9" y2="40.64" width="0.4064" layer="1"/>
+<wire x1="88.9" y1="40.64" x2="86.36" y2="38.1" width="0.4064" layer="1"/>
 </signal>
 <signal name="N$17">
@@
 <signal name="N$3">
 <contactref element="IC2" pad="3"/>
-<contactref element="RV2" pad="3"/>
-<wire x1="28.16723125" y1="45.72" x2="21.0312" y2="38.58396875" width="0.4064" layer="1"/>
-<wire x1="21.0312" y1="38.58396875" x2="21.0312" y2="35.07603125" width="0.4064" layer="1"/>
-<wire x1="21.0312" y1="35.07603125" x2="21.81723125" y2="34.29" width="0.4064" layer="1"/>
-<wire x1="21.81723125" y1="34.29" x2="23.90276875" y2="34.29" width="0.4064" layer="1"/>
-<wire x1="23.90276875" y1="34.29" x2="24.6888" y2="33.50396875" width="0.4064" layer="1"/>
-<wire x1="24.6888" y1="33.50396875" x2="24.6888" y2="29.7688" width="0.4064" layer="1"/>
-<wire x1="24.6888" y1="29.7688" x2="22.86" y2="27.94" width="0.4064" layer="1"/>
-<wire x1="38.18" y1="50.8" x2="33.1" y2="45.72" width="0.4064" layer="1"/>
-<wire x1="33.1" y1="45.72" x2="28.16723125" y2="45.72" width="0.4064" layer="1"/>
+<contactref element="RV2" pad="2"/>
+<wire x1="43.18" y1="50.8" x2="39.37" y2="46.99" width="0.4064" layer="1"/>
+<wire x1="39.37" y1="46.99" x2="36.83" y2="46.99" width="0.4064" layer="1"/>
+<wire x1="33.655" y1="43.815" x2="33.655" y2="41.275" width="0.4064" layer="1"/>
+<wire x1="33.655" y1="41.275" x2="33.02" y2="40.64" width="0.4064" layer="1"/>
+<wire x1="19.304" y1="37.973" x2="19.304" y2="30.099" width="0.4064" layer="1"/>
+<wire x1="19.304" y1="30.099" x2="19.232140625" y2="30.170859375" width="0.4064" layer="1"/>
+<wire x1="19.232140625" y1="30.170859375" x2="19.232140625" y2="30.281140625" width="0.4064" layer="1"/>
+<via x="19.232140625" y="30.281140625" extent="1-16" drill="0.35"/>
+<wire x1="19.232140625" y1="30.281140625" x2="19.248859375" y2="30.281140625" width="0.4064" layer="16"/>
+<wire x1="36.83" y1="46.99" x2="33.655" y2="43.815" width="0.4064" layer="1"/>
+<wire x1="33.02" y1="40.64" x2="21.971" y2="40.64" width="0.4064" layer="1"/>
+<wire x1="21.971" y1="40.64" x2="19.304" y2="37.973" width="0.4064" layer="1"/>
+<wire x1="21.59" y1="27.94" x2="22.86" y2="27.94" width="0.4064" layer="16"/>
+<wire x1="19.248859375" y1="30.281140625" x2="21.59" y2="27.94" width="0.4064" layer="16"/>
 </signal>
 <signal name="N$22">
@@
 <signal name="N$24">
 <contactref element="R7" pad="1"/>
-<contactref element="RV2" pad="2"/>
+<contactref element="RV2" pad="3"/>
 <contactref element="J1" pad="P$3"/>
 <wire x1="29.18" y1="45.75" x2="31.75" y2="43.18" width="0.4064" layer="16"/>
 <wire x1="20.32" y1="48.27" x2="22.84" y2="45.75" width="0.4064" layer="16"/>
 <wire x1="22.84" y1="45.75" x2="29.18" y2="45.75" width="0.4064" layer="16"/>
-<wire x1="33.985196875" y1="45.415196875" x2="31.75" y2="43.18" width="0.4064" layer="1"/>
-<wire x1="35.255196875" y1="45.415196875" x2="33.985196875" y2="45.415196875" width="0.4064" layer="1"/>
-<wire x1="43.18" y1="50.8" x2="40.64" y2="50.8" width="0.4064" layer="1"/>
-<wire x1="40.64" y1="50.8" x2="35.255196875" y2="45.415196875" width="0.4064" layer="1"/>
+<wire x1="38.18" y1="50.8" x2="31.75" y2="44.37" width="0.4064" layer="1"/>
+<wire x1="31.75" y1="44.37" x2="31.75" y2="43.18" width="0.4064" layer="1"/>
 </signal>
 <signal name="N$2">
@@
 </drawing>
 <compatibility>
-<note version="6.3" minversion="6.2.2" severity="warning">
-Since Version 6.2.2 text objects can contain more than one line,
-which will not be processed correctly with this version.
-</note>
 <note version="8.2" severity="warning">
 Since Version 8.2, EAGLE supports online libraries. The ids
