File: v2.0/schematics/eagle/mixer.rev1/mixer-board1.brd (EAGLE design)
At the start: 100 x 80 mm, 8 parts

Commit message: Added input stage to mixer
Parts:
- added C1, C10, C11, C12, C13, C14, C18, C19, C2, C20, C4, C9: 47uF, _common:E2-5
- added C15, C16, C17, C3, C5, C6, C7, C8: 20pF, _common:C025-024X044
- added IC1, IC2: TL084P, _common:DIL14
- added R1, R17, R18, R19, R2, R20, R21, R22: 100K, _common:0207/7
- added R10, R11, R6, R9: 2.7K, _common:0207/7
- added R12, R13, R14, R26, R27, R31, R5, R7, R8: 5.1K, _common:0207/7
- added R15, R16: 10K, _common:0207/7
- added R23, R24, R25, R3: 1K, _common:0207/7
- added R28, R29, R30, R4: 510, _common:0207/7
- J1: value (none) -> M1
- J2: value (none) -> M2
- J3: value (none) -> SEND1
- J4: value (none) -> SEND2
- J5: value (none) -> ST1-L
- J6: value (none) -> ST1-R
- J7: value (none) -> ST2-L
- J8: value (none) -> ST2-R
Connections:
- new net 0V: IC2.10, IC2.12, IC2.3, IC2.5, J1.P$1, J1.P$2, J1.P$3, J3.P$1, J3.P$2, J3.P$3, R15.1, R16.1, R2.1, R21.1, R29.1, R4.1
- new net FX-MX-1: R31.2
- new net M1-LVL-2: R1.1
- new net M1-LVL-3: C1.-
- new net N$1: C1.+, J1.P$4
- new net N$10: R13.1, R14.1
- new net N$11: C7.1, IC2.8, R11.1, R9.2
- new net N$12: C8.2, IC2.13, R11.2, R8.1
- new net N$13: C6.1, C9.-, IC2.7, R7.2
- new net N$14: C12.+, J3.P$4
- new net N$15: C7.2, IC2.9, R12.2, R14.2, R9.1
- new net N$16: C12.-, R18.1
- new net N$17: IC1.10, R18.2, R21.2
- new net N$18: C10.-, C8.1, IC2.14, R8.2
- new net N$19: C16.2, IC1.9, R24.1, R29.2
- new net N$2: C3.2, IC1.2, R3.1, R4.2
- new net N$20: C16.1, C19.+, IC1.8, R24.2
- new net N$21: C19.-, R26.1, R31.1
- new net N$3: C2.-, IC1.3, R2.2
- new net N$4: C2.+, R1.2
- new net N$5: C3.1, C4.+, IC1.1, R3.2
- new net N$6: C4.-, R12.1, R5.1
- new net N$7: C5.2, IC2.2, R13.2, R5.2, R6.1
- new net N$8: C5.1, IC2.1, R10.1, R6.2
- new net N$9: C6.2, IC2.6, R10.2, R7.1
- new net OUT-LVL-3: C9.+, R15.2
- new net OUT-LVL-6: C10.+, R16.2
- new net SEND1-OUT: R26.2
- new net V+: IC1.4, IC2.4
- new net V-: IC1.11, IC2.11

Commit message: Update final amp stage value to line level
Parts:
- R7: value 5.1K -> 2.7K
Changed lines of the file:
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@@
 <attribute name="VALUE" x="2.794" y="-169.4688" size="1.27" layer="27" ratio="10"/>
 </element>
-<element name="R7" library="_common" package="0207/7" value="5.1K" x="5.08" y="-173.99" smashed="yes">
+<element name="R7" library="_common" package="0207/7" value="2.7K" x="5.08" y="-173.99" smashed="yes">
 <attribute name="NAME" x="2.54" y="-172.593" size="1.27" layer="25" ratio="10"/>
 <attribute name="VALUE" x="2.794" y="-174.5488" size="1.27" layer="27" ratio="10"/>

Commit message: Updated caps to 100uF
Parts:
- C1, C10, C11, C12, C13, C14, C18, C19, C2, C20, C4, C9: value 47uF -> 100uF
Changed lines of the file:
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@@
 <attribute name="VALUE" x="3.74" y="-88.35" size="1.27" layer="27"/>
 </element>
-<element name="C1" library="_common" package="E2-5" value="47uF" x="3.81" y="-93.98" smashed="yes">
+<element name="C1" library="_common" package="E2-5" value="100uF" x="3.81" y="-93.98" smashed="yes">
 <attribute name="NAME" x="6.35" y="-92.964" size="1.27" layer="25" ratio="10"/>
 <attribute name="VALUE" x="6.35" y="-96.139" size="1.27" layer="27" ratio="10"/>
@@
 <attribute name="VALUE" x="2.794" y="-117.3988" size="1.27" layer="27" ratio="10"/>
 </element>
-<element name="C2" library="_common" package="E2-5" value="47uF" x="3.81" y="-121.92" smashed="yes">
+<element name="C2" library="_common" package="E2-5" value="100uF" x="3.81" y="-121.92" smashed="yes">
 <attribute name="NAME" x="6.35" y="-120.904" size="1.27" layer="25" ratio="10"/>
 <attribute name="VALUE" x="6.35" y="-124.079" size="1.27" layer="27" ratio="10"/>
@@
 <attribute name="VALUE" x="2.794" y="-141.5288" size="1.27" layer="27" ratio="10"/>
 </element>
-<element name="C4" library="_common" package="E2-5" value="47uF" x="3.81" y="-146.05" smashed="yes">
+<element name="C4" library="_common" package="E2-5" value="100uF" x="3.81" y="-146.05" smashed="yes">
 <attribute name="NAME" x="6.35" y="-145.034" size="1.27" layer="25" ratio="10"/>
 <attribute name="VALUE" x="6.35" y="-148.209" size="1.27" layer="27" ratio="10"/>
@@
 <attribute name="VALUE" x="2.794" y="-240.5888" size="1.27" layer="27" ratio="10"/>
 </element>
-<element name="C9" library="_common" package="E2-5" value="47uF" x="3.81" y="-245.11" smashed="yes">
+<element name="C9" library="_common" package="E2-5" value="100uF" x="3.81" y="-245.11" smashed="yes">
 <attribute name="NAME" x="6.35" y="-244.094" size="1.27" layer="25" ratio="10"/>
 <attribute name="VALUE" x="6.35" y="-247.269" size="1.27" layer="27" ratio="10"/>
 </element>
-<element name="C10" library="_common" package="E2-5" value="47uF" x="3.81" y="-251.46" smashed="yes">
+<element name="C10" library="_common" package="E2-5" value="100uF" x="3.81" y="-251.46" smashed="yes">
 <attribute name="NAME" x="6.35" y="-250.444" size="1.27" layer="25" ratio="10"/>
 <attribute name="VALUE" x="6.35" y="-253.619" size="1.27" layer="27" ratio="10"/>
@@
 <attribute name="VALUE" x="2.794" y="-263.4488" size="1.27" layer="27" ratio="10"/>
 </element>
-<element name="C11" library="_common" package="E2-5" value="47uF" x="3.81" y="-267.97" smashed="yes">
+<element name="C11" library="_common" package="E2-5" value="100uF" x="3.81" y="-267.97" smashed="yes">
 <attribute name="NAME" x="6.35" y="-266.954" size="1.27" layer="25" ratio="10"/>
 <attribute name="VALUE" x="6.35" y="-270.129" size="1.27" layer="27" ratio="10"/>
 </element>
-<element name="C12" library="_common" package="E2-5" value="47uF" x="3.81" y="-274.32" smashed="yes">
+<element name="C12" library="_common" package="E2-5" value="100uF" x="3.81" y="-274.32" smashed="yes">
 <attribute name="NAME" x="6.35" y="-273.304" size="1.27" layer="25" ratio="10"/>
 <attribute name="VALUE" x="6.35" y="-276.479" size="1.27" layer="27" ratio="10"/>
 </element>
-<element name="C13" library="_common" package="E2-5" value="47uF" x="3.81" y="-280.67" smashed="yes">
+<element name="C13" library="_common" package="E2-5" value="100uF" x="3.81" y="-280.67" smashed="yes">
 <attribute name="NAME" x="6.35" y="-279.654" size="1.27" layer="25" ratio="10"/>
 <attribute name="VALUE" x="6.35" y="-282.829" size="1.27" layer="27" ratio="10"/>
@@
 <attribute name="VALUE" x="2.794" y="-312.9788" size="1.27" layer="27" ratio="10"/>
 </element>
-<element name="C14" library="_common" package="E2-5" value="47uF" x="3.81" y="-317.5" smashed="yes">
+<element name="C14" library="_common" package="E2-5" value="100uF" x="3.81" y="-317.5" smashed="yes">
 <attribute name="NAME" x="6.35" y="-316.484" size="1.27" layer="25" ratio="10"/>
 <attribute name="VALUE" x="6.35" y="-319.659" size="1.27" layer="27" ratio="10"/>
@@
 <attribute name="VALUE" x="0.762" y="-356.997" size="1.27" layer="27" ratio="10"/>
 </element>
-<element name="C18" library="_common" package="E2-5" value="47uF" x="3.81" y="-360.68" smashed="yes">
+<element name="C18" library="_common" package="E2-5" value="100uF" x="3.81" y="-360.68" smashed="yes">
 <attribute name="NAME" x="6.35" y="-359.664" size="1.27" layer="25" ratio="10"/>
 <attribute name="VALUE" x="6.35" y="-362.839" size="1.27" layer="27" ratio="10"/>
 </element>
-<element name="C19" library="_common" package="E2-5" value="47uF" x="3.81" y="-367.03" smashed="yes">
+<element name="C19" library="_common" package="E2-5" value="100uF" x="3.81" y="-367.03" smashed="yes">
 <attribute name="NAME" x="6.35" y="-366.014" size="1.27" layer="25" ratio="10"/>
 <attribute name="VALUE" x="6.35" y="-369.189" size="1.27" layer="27" ratio="10"/>
 </element>
-<element name="C20" library="_common" package="E2-5" value="47uF" x="3.81" y="-373.38" smashed="yes">
+<element name="C20" library="_common" package="E2-5" value="100uF" x="3.81" y="-373.38" smashed="yes">
 <attribute name="NAME" x="6.35" y="-372.364" size="1.27" layer="25" ratio="10"/>
 <attribute name="VALUE" x="6.35" y="-375.539" size="1.27" layer="27" ratio="10"/>

Commit message: Added stereo line in; output level
Parts:
- R7: value 2.7K -> 5.1K
Changed lines of the file:
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@@
 <attribute name="VALUE" x="2.794" y="-169.4688" size="1.27" layer="27" ratio="10"/>
 </element>
-<element name="R7" library="_common" package="0207/7" value="2.7K" x="5.08" y="-173.99" smashed="yes">
+<element name="R7" library="_common" package="0207/7" value="5.1K" x="5.08" y="-173.99" smashed="yes">
 <attribute name="NAME" x="2.54" y="-172.593" size="1.27" layer="25" ratio="10"/>
 <attribute name="VALUE" x="2.794" y="-174.5488" size="1.27" layer="27" ratio="10"/>

Commit message: Completed initial mixer schematic draft
Parts:
- added C21, C22, C23, C24, C31, C32, C33, C34, C35, C36, C41, C42, C43, C44: 100uF, _common:E2-5
- added C25, C26, C27, C28, C29, C30, C37, C38, C39, C40: 22pF, _common:C025-024X044
- added IC3, IC4: TL082P, _common:DIL08
- added JP1: PWR, pinhead:2X05
- added JP2, JP4: (no value), pinhead:2X08
- added JP3, JP5: (no value), pinhead:2X05
- added R32, R33, R34, R35, R36, R37, R38, R43, R44: 5.1K, _common:0207/7
- added R39, R40, R41, R42: 2.7K, _common:0207/7
- added R45, R46: 10K, _common:0207/7
- C1, C2: value 100uF -> 10uF; device _common:E2-5 -> _common.v1:E2-5
- C10, C11, C12, C4, C9: value 100uF -> 0.1uF; device _common:E2-5 -> _common.v1:C025-024X044
- C15, C16, C17: value 20pF -> 100uF; device _common:C025-024X044 -> _common:E2-5
- C3, C5, C6, C7, C8: value 20pF -> 0.1uF; device _common:C025-024X044 -> _common.v1:C025-024X044
- IC1: value TL084P -> TL082P; device _common:DIL14 -> _common:DIL08
- J1: value M1 -> M2
- J2: value M2 -> ST1-L
- J3: value SEND1 -> ST1-R
- J4: value SEND2 -> ST2-L
- J5: value ST1-L -> ST2-R
- J6: value ST1-R -> M1
- J7: value ST2-L -> SEND1
- J8: value ST2-R -> SEND2
- R10, R11, R6, R9: value 2.7K -> 100K
- R12, R5, R7, R8: value 5.1K -> 100K
- R13, R14: value 5.1K -> 510
- R15, R16: value 10K -> 510
- R17, R18: value 100K -> 510
- R19, R20, R21, R22: value 100K -> 1K
- R25: value 1K -> 5.1K
- R28, R29, R30: value 510 -> 5.1K
- R3: value 1K -> 100K
- R4: value 510 -> 100K
- moved IC1 552.5 mm to (7.62, -660.4)
- moved R6 449.6 mm to (5.08, -618.5)
- moved R5 431.8 mm to (5.08, -584.2)
- moved R4 408.9 mm to (5.08, -549.9)
- moved R12 388.8 mm to (15.2, -618.5)
- moved R3 382.4 mm to (15.2, -510.5)
- moved C1 378.5 mm to (8.89, -472.4)
- moved R11 359.6 mm to (15.2, -584.2)
- moved C2 358.1 mm to (3.81, -480.1)
- moved R18 331.6 mm to (15.2, -623.6)
- moved R9 331.5 mm to (5.08, -515.6)
- moved R10 330.4 mm to (15.2, -549.9)
- moved C3 317.5 mm to (2.54, -450.9)
- moved C4 304.8 mm to (8.89, -450.9)
- moved R17 302.4 mm to (15.2, -589.3)
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Connections:
- removed net FX-MX-1: R31.2
- removed net N$16: C12.-, R18.1
- removed net N$17: IC1.10, R18.2, R21.2
- removed net N$19: C16.2, IC1.9, R24.1, R29.2
- removed net N$20: C16.1, C19.+, IC1.8, R24.2
- removed net N$21: C19.-, R26.1, R31.1
- removed net SEND1-OUT: R26.2
- removed net V+: IC1.4, IC2.4
- removed net V-: IC1.11, IC2.11
- new net +12V: C1.+, C11.1, C3.1, C5.1, C7.1, C9.1, IC1.8, IC2.4, IC3.8, IC4.8, JP1.10, JP1.9, JP4.5, JP5.5
- new net -12V: C10.2, C12.2, C2.-, C4.2, C6.2, C8.2, IC1.4, IC2.11, IC3.4, IC4.4, JP1.1, JP1.2, JP4.1, JP5.1
- new net FX1-1-SEND1: C41.-, JP3.1, JP4.11
- new net FX1-2-MIX-L: JP3.3, R35.1
- new net FX1-3-RTN1-L: JP3.5, JP4.2
- new net FX1-5-MIX-R: JP3.7, R36.1
- new net FX1-6-RTN1-R: JP3.9, JP4.4
- new net FX2-1-SEND2: C42.-, JP3.2, JP4.13
- new net FX2-2-MIX-L: JP3.4, R37.1
- new net FX2-3-RTN2-L: JP3.6, JP4.6
- new net FX2-5-MIX-R: JP3.8, R38.1
- new net FX2-6-RTN2-R: JP3.10, JP4.8
- new net M2-LVL-2: JP4.9, R2.1
- new net M2-LVL-3: C14.-, JP4.7
- new net N$22: C26.1, C32.+, IC1.7, R20.2
- new net N$23: C26.2, IC1.6, R14.2, R20.1
- new net N$24: C20.-, IC1.5, R8.2
- new net N$25: C20.+, R2.2
- new net N$26: C14.+, J1.P$4
- new net N$28: C34.-, R30.1
- new net N$29: C33.-, R29.1
- new net N$30: C27.1, C33.+, IC2.1, R21.2
- new net N$31: C27.2, IC2.2, R15.2, R21.1
- new net N$32: C21.-, IC2.3, R9.2
- new net N$33: C21.+, R3.2
- new net N$34: C15.+, J2.P$4
- new net N$35: C28.1, C34.+, IC2.7, R22.2
- new net N$36: C28.2, IC2.6, R16.2, R22.1
- new net N$37: C22.-, IC2.5, R10.2
- new net N$38: C22.+, R4.2
- new net N$39: C16.+, J3.P$4
- new net N$41: C35.-, R31.1
- new net N$42: C29.1, C35.+, IC2.8, R23.2
- new net N$43: C29.2, IC2.9, R17.2, R23.1
- new net N$44: C23.-, IC2.10, R11.2
- new net N$45: C23.+, R5.2
- new net N$46: C17.+, J4.P$4
- new net N$48: C36.-, R32.1
- new net N$49: C30.1, C36.+, IC2.14, R24.2
- new net N$50: C30.2, IC2.13, R18.2, R24.1
- new net N$51: C24.-, IC2.12, R12.2
- new net N$52: C24.+, R6.2
- new net N$53: C18.+, J5.P$4
- new net N$58: C42.+, J8.P$4
- new net ST1-LVL-2: R3.1
- new net ST1-LVL-3: C15.-, JP2.7
- new net ST1-LVL-5: JP2.13, R4.1
- new net ST1-LVL-6: C16.-, JP2.11
- new net ST1-LVL2: JP2.9
- new net ST2-LVL-2: JP2.10, R5.1
- new net ST2-LVL-3: C17.-, JP2.8
- new net ST2-LVL-5: JP2.14, R6.1
- new net ST2-LVL-6: C18.-, JP2.12
- new net ST3-L: JP5.7, R33.1
- new net ST3-R: JP5.9, R34.1
- net 0V: now also C1.-, C10.1, C11.2, C12.1, C2.+, C3.2, C4.1, C5.2, C6.1, C7.2, C8.1, C9.2, IC3.3, IC3.5, IC4.3, IC4.5, J2.P$1, J2.P$2, J2.P$3, J4.P$1, J4.P$2, J4.P$3, J5.P$1, J5.P$2, J5.P$3, J6.P$1, J6.P$2, J6.P$3, J7.P$1, J7.P$2, J7.P$3, J8.P$1, J8.P$2, J8.P$3, JP1.3, JP1.4, JP1.5, JP1.6, JP1.7, JP1.8, JP2.1, JP2.15, JP2.16, JP2.2, JP4.3, JP5.3, R10.1, R11.1, R12.1, R13.1, R14.1, R17.1, R18.1, R45.1, R46.1, R7.1, R8.1, R9.1; no longer IC2.10, IC2.12, IC2.3, IC2.5, R2.1, R21.1, R29.1, R4.1
- net M1-LVL-2: now also JP2.5
- net M1-LVL-3: now also C13.-, JP2.3; no longer C1.-
- net N$1: now also C13.+, J6.P$4; no longer C1.+, J1.P$4
- net N$10: now also C32.-, R27.1, R28.1; no longer R13.1, R14.1
- net N$11: now also C38.1, IC4.1, R40.2, R42.1; no longer C7.1, IC2.8, R11.1, R9.2
- net N$12: now also C40.2, IC4.6, R42.2, R44.1; no longer C8.2, IC2.13, R11.2, R8.1
- net N$13: now also C39.1, C43.-, IC3.7, R43.2; no longer C6.1, C9.-, IC2.7, R7.2
- net N$14: now also C41.+, J7.P$4; no longer C12.+, J3.P$4
- net N$15: now also C38.2, IC4.2, R26.2, R28.2, R30.2, R32.2, R34.2, R36.2, R38.2, R40.1; no longer C7.2, IC2.9, R12.2, R14.2, R9.1
- net N$18: now also C40.1, C44.-, IC4.7, R44.2; no longer C10.-, C8.1, IC2.14, R8.2
- net N$2: now also C25.2, R13.2, R19.1; no longer C3.2, R3.1, R4.2
- net N$3: now also C19.-, R7.2; no longer C2.-, R2.2
- net N$4: now also C19.+; no longer C2.+
- net N$5: now also C25.1, C31.+, R19.2; no longer C3.1, C4.+, R3.2
- net N$6: now also C31.-, R25.1, R26.1; no longer C4.-, R12.1, R5.1
- net N$7: now also C37.2, IC3.2, R25.2, R27.2, R29.2, R31.2, R33.2, R35.2, R37.2, R39.1; no longer C5.2, IC2.2, R13.2, R5.2, R6.1
- net N$8: now also C37.1, IC3.1, R39.2, R41.1; no longer C5.1, IC2.1, R10.1, R6.2
- net N$9: now also C39.2, IC3.6, R41.2, R43.1; no longer C6.2, IC2.6, R10.2, R7.1
- net OUT-LVL-3: now also C43.+, JP5.2, R45.2; no longer C9.+, R15.2
- net OUT-LVL-6: now also C44.+, JP5.4, R46.2; no longer C10.+, R16.2

Commit message: Fixed jack grounds; normalled R to L; increased master gain
Connections:
- removed net N$26: C14.+, J1.P$4
- removed net N$34: C15.+, J2.P$4
- removed net N$39: C16.+, J3.P$4
- removed net N$46: C17.+, J4.P$4
- removed net N$53: C18.+, J5.P$4
- removed net N$58: C42.+, J8.P$4
- new net N$16: C14.+, J1.P$3
- new net N$17: C15.+, J2.P$3, J3.P$4
- new net N$19: C16.+, J3.P$3
- new net N$20: C17.+, J4.P$3, J5.P$4
- new net N$21: C18.+, J5.P$3
- new net N$27: C41.+, J7.P$3
- net 0V: now also J1.P$4, J2.P$4, J4.P$4, J6.P$4, J7.P$4, J8.P$4; no longer J1.P$3, J2.P$3, J3.P$3, J4.P$3, J5.P$3, J6.P$3, J7.P$3, J8.P$3
- net N$1: now also J6.P$3; no longer J6.P$4
- net N$14: now also C42.+, J8.P$3; no longer C41.+, J7.P$4

Commit message: Updated VAR-ST; Added FX Crossfades; Ran error checks
Parts:
- removed R45, R46: 10K, _common:0207/7
- JP1: value PWR -> BOARD2-A; device pinhead:2X05 -> pinhead:2X08
- JP2: value (none) -> BOARD2-B; device pinhead:2X08 -> pinhead:2X05
- JP3: value (none) -> BOARD3; device pinhead:2X05 -> pinhead:2X08
- JP4: value (none) -> BOARD4; device pinhead:2X08 -> pinhead:2X05
- JP5: value (none) -> PWR
- R37, R38: value 5.1K -> 2.7K
- R41, R42: value 2.7K -> 5.1K
- R43, R44: value 5.1K -> 10K
- moved R37 525.8 mm to (5.08, -168.9)
- moved R38 515.6 mm to (5.08, -184.2)
- moved JP2 292.1 mm to (7.62, -703.6)
- moved JP1 254.0 mm to (11.4, -696.0)
- moved R43 83.8 mm to (5.08, -257.8)
- moved R44 83.8 mm to (5.08, -262.9)
- moved R39 50.8 mm to (5.08, -219.7)
- moved R41 45.7 mm to (5.08, -174.0)
- moved R42 45.7 mm to (5.08, -179.1)
- moved R40 40.6 mm to (5.08, -224.8)
- moved JP3 8.52 mm to (11.4, -426.7)
- moved JP4 8.52 mm to (7.62, -434.3)
- moved JP5 7.62 mm to (7.62, -442.0)
Connections:
- removed net FX1-1-SEND1: C41.-, JP3.1, JP4.11
- removed net FX1-2-MIX-L: JP3.3, R35.1
- removed net FX1-3-RTN1-L: JP3.5, JP4.2
- removed net FX1-5-MIX-R: JP3.7, R36.1
- removed net FX1-6-RTN1-R: JP3.9, JP4.4
- removed net FX2-1-SEND2: C42.-, JP3.2, JP4.13
- removed net FX2-2-MIX-L: JP3.4, R37.1
- removed net FX2-3-RTN2-L: JP3.6, JP4.6
- removed net FX2-5-MIX-R: JP3.8, R38.1
- removed net FX2-6-RTN2-R: JP3.10, JP4.8
- removed net ST1-LVL2: JP2.9
- new net FX-MIX-L: JP2.7, R35.1
- new net FX-MIX-R: JP2.9, R36.1
- new net FX1-RTN-L: JP2.2, JP3.2
- new net FX1-RTN-R: JP2.4, JP3.4
- new net FX1-SEND: C41.-, JP2.3, JP3.11
- new net FX2-RTN-L: JP2.6, JP3.6
- new net FX2-RTN-R: JP2.8, JP3.8
- new net FX2-SEND: C42.-, JP2.5, JP3.13
- net +12V: now also JP1.5, JP3.5, JP5.10, JP5.9; no longer JP1.10, JP1.9, JP5.5
- net -12V: now also JP3.1, JP5.2; no longer JP1.2
- net 0V: now also JP1.14, JP2.10, JP3.14, JP3.3, JP4.8, JP5.4, JP5.5, JP5.6, JP5.7, JP5.8, R43.1, R44.1; no longer JP1.4, JP1.5, JP1.6, JP1.7, JP1.8, JP2.15, JP2.16, JP2.2, R45.1, R46.1
- net M1-LVL-2: now also JP1.10; no longer JP2.5
- net M1-LVL-3: now also JP1.7; no longer JP2.3
- net M2-LVL-2: now also JP3.9; no longer JP4.9
- net M2-LVL-3: now also JP3.7; no longer JP4.7
- net N$11: now also R38.2, R40.1; no longer R40.2, R42.1
- net N$12: now also R40.2, R42.1; no longer R42.2, R44.1
- net N$13: now also R41.2; no longer R43.2
- net N$15: now also R38.1; no longer R38.2, R40.1
- net N$18: now also R42.2; no longer R44.2
- net N$7: now also R37.1; no longer R37.2, R39.1
- net N$8: now also R37.2, R39.1; no longer R39.2, R41.1
- net N$9: now also R39.2, R41.1; no longer R41.2, R43.1
- net OUT-LVL-3: now also JP4.2, R43.2; no longer JP5.2, R45.2
- net OUT-LVL-6: now also JP4.4, R44.2; no longer JP5.4, R46.2
- net ST1-LVL-2: now also JP1.11
- net ST1-LVL-3: now also JP1.9; no longer JP2.7
- net ST1-LVL-5: now also JP1.15; no longer JP2.13
- net ST1-LVL-6: now also JP1.13; no longer JP2.11
- net ST2-LVL-2: now also JP1.4; no longer JP2.10
- net ST2-LVL-3: now also JP1.2; no longer JP2.8
- net ST2-LVL-5: now also JP1.8; no longer JP2.14
- net ST2-LVL-6: now also JP1.6; no longer JP2.12
- net ST3-L: now also JP4.7; no longer JP5.7
- net ST3-R: now also JP4.9; no longer JP5.9

Commit message: Updated cap packages
Parts:
- C1, C2: value 10uF -> 100uF; device _common.v1:E2-5 -> _common:E5-8,5
- C13, C14, C15, C16, C17, C18, C19, C20, C21, C22, C23, C24, C31, C32, C33, C34, C35, C36, C41, C42, C43, C44: device _common:E2-5 -> _common:E5-8,5
- moved C13 623.6 mm to (-2.54, -717.5)
- moved C19 608.4 mm to (-2.54, -730.2)
- moved C31 596.9 mm to (-2.54, -743.0)
- moved C14 538.5 mm to (-2.54, -806.5)
- moved C2 529.6 mm to (-2.54, -1009.6)
- moved C1 524.6 mm to (-2.54, -997.0)
- moved C44 516.9 mm to (-2.54, -768.4)
- moved C43 510.6 mm to (-2.54, -755.6)
- moved C42 496.6 mm to (-2.54, -870.0)
- moved C41 490.3 mm to (-2.54, -857.2)
- moved C20 476.3 mm to (-2.54, -793.8)
- moved C32 420.4 mm to (-2.54, -781.0)
- moved C18 378.5 mm to (-2.54, -984.2)
- moved C16 370.9 mm to (-2.54, -908.0)
- moved C35 368.4 mm to (-2.54, -946.1)
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